File: PCB/CTRL/CTRL.kicad_pcb (KiCad board)
At the start: 2 copper layers, 40 x 46.2 mm, 11 parts, among them J1 Conn_02x06_Odd_Even, J2 Conn_02x06_Odd_Even, U3 MAX6372

Commit message: udated by FZ
Parts:
- removed C10: 0.1uF, Capacitor_SMD:C_0402_1005Metric
- removed C9: 47uF, Capacitor_SMD:C_0805_2012Metric_Pad1.18x1.45mm_HandSolder
- removed JP1: RST Jumper, Jumper:SolderJumper-3_P1.3mm_Open_RoundedPad1.0x1.5mm
- removed R5, R6: 27, Resistor_SMD:R_0402_1005Metric_Pad0.72x0.64mm_HandSolder
- removed U3: MAX6372, Package_TO_SOT_SMD:SOT-23-8
- added C2: 10uF, Capacitor_SMD:C_1206_3216Metric_Pad1.33x1.80mm_HandSolder, F.Cu at (155.7, 91.6)
- added C3: 10uF, Capacitor_SMD:C_1206_3216Metric_Pad1.33x1.80mm_HandSolder, F.Cu at (153.3, 91.6)
- added C4: 0.1uF, Capacitor_SMD:C_0402_1005Metric_Pad0.74x0.62mm_HandSolder, F.Cu at (155.2, 110.3)
- added D1: LED, Diode_SMD:D_0603_1608Metric_Pad1.05x0.95mm_HandSolder, B.Cu at (164.7, 99.2)
- added F1: Fuse_Small, Fuse:Fuse_1206_3216Metric_Pad1.42x1.75mm_HandSolder, F.Cu at (158.2, 91.6)
- added J3: USB3131-30-0230-A_REVB, Mylib:GCT_USB3131-30-0230-A_REVB, B.Cu at (157.8, 100.1)
- added J4: RESET, Connector_PinHeader_2.00mm:PinHeader_1x02_P2.00mm_Vertical, F.Cu at (131.9, 103.7)
- added J5: RESET, Connector_PinHeader_2.00mm:PinHeader_1x02_P2.00mm_Vertical, F.Cu at (131.9, 95.0)
- added J6: Conn_01x04_Pin, Connector_PinHeader_2.00mm:PinHeader_1x04_P2.00mm_Vertical, F.Cu at (168.6, 97.1)
- added R1: 27, Resistor_SMD:R_0402_1005Metric_Pad0.72x0.64mm_HandSolder, F.Cu at (165.6, 99.1)
- added R14: 15K, Resistor_SMD:R_0402_1005Metric_Pad0.72x0.64mm_HandSolder, F.Cu at (165.6, 102.1)
- added R15: 15K, Resistor_SMD:R_0402_1005Metric_Pad0.72x0.64mm_HandSolder, F.Cu at (165.6, 98.0)
- added R2: 27, Resistor_SMD:R_0402_1005Metric_Pad0.72x0.64mm_HandSolder, F.Cu at (165.6, 101.1)
- added R3: 330, Resistor_SMD:R_0402_1005Metric_Pad0.72x0.64mm_HandSolder, F.Cu at (153.4, 110.9)
- added S1: TL1105F160Q, Mylib:SW_TL1105F160Q, B.Cu at (141.2, 99.9)
- added S2: SS12D07VG4, Mylib:SW_SS12D07VG4, B.Cu at (150.2, 97.2)
- added S3: SS12D07VG4, Mylib:SW_SS12D07VG4, B.Cu at (150.2, 102.7)
- added TP3: TestPoint, TestPoint:TestPoint_Pad_1.5x1.5mm, F.Cu at (163.6, 86.9)
- added U4: SN65220DBVR, SamacSys_Parts:SOT95P275X135-6N, F.Cu at (162.2, 100.1)
- R4: value 10K -> 1M; footprint Resistor_SMD:R_0402_1005Metric -> Resistor_SMD:R_0603_1608Metric_Pad0.98x0.95mm_HandSolder
- TP1: value VCC_TP -> TestPoint; moved to B.Cu
- TP2: value GND_TP -> TestPoint
- moved TP2 23.2 mm to (160.2, 84.9), turned to 150 degrees
- moved R4 16.5 mm to (151.3, 91.0), turned to 90 degrees
- moved TP1 8.38 mm to (140.9, 93.3), turned to 180 degrees
Connections:
- net /D11 renamed /D12
- net /D6 renamed /D1
- net /LED2 renamed /D4
- net /VBAT_OK renamed /A3
- net /~{CS} renamed /A4
- net /~{EN} renamed /D8
- J1 pad 3: VCC -> /A5
- J1 pad 5: /~{I2C_RESET} -> +5V
- J1 pad 6: +5V -> /A2
- J2 pad 2: /D13 -> /D10
- J2 pad 3: /A1 -> /MOSI
- J2 pad 6: /A5 -> /D3
- J2 pad 7: /MOSI -> /D2
- R4 pad 1: /D2 -> GND
- R4 pad 2: GND -> +5V
- TP1 pad 1: VCC -> /VBAT
- TP2 pad 1: GND -> Net-(D1-K)
Routing:
- net +5V: track 0.05 -> 24.8 mm
- net Net-(J5-Pin_2): track 0.00 -> 24.4 mm
- net Net-(J5-Pin_1): track 0.00 -> 22.6 mm
- net /LORA_FREQ_SELECT: track 0.00 -> 22.4 mm
- net Net-(D1-K): track 0.00 -> 15.8 mm, vias 0 -> 1
- net Net-(D1-A): track 0.00 -> 14.3 mm, vias 0 -> 1
- net Net-(J4-Pin_2): track 0.00 -> 12.1 mm
- net Net-(J3-VCC): track 0.00 -> 12.1 mm
- net /USB-: track 0.00 -> 11.3 mm, vias 0 -> 1
- net /D10: track 0.00 -> 9.82 mm
- net /USB+: track 0.00 -> 9.15 mm
- net /VBAT: track 0.00 -> 8.03 mm
- net Net-(J4-Pin_1): track 0.00 -> 7.17 mm
- net GND: track 0.00 -> 4.80 mm, vias 17 -> 129
- net Net-(J6-Pin_3): track 0.00 -> 2.40 mm
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Other:
- board text added: "868MHz"
- board text added: "915MHz"
- board text added: "OFF"
- board text added: "ON"
- board text removed: "X"
- board text removed: "Y"
- board text removed: "Z"
