File: PCB/MCU/MCU.kicad_pcb (KiCad board)
At the start: 2 copper layers, 40 x 46.2 mm, 57 parts, among them IC2 LTC4311CSC6#TRPBF, J1 Conn_02x06_Odd_Even, J2 Conn_02x06_Odd_Even, J4 Conn_01x04_Pin, J5 RESET, J6 Conn_01x04_Pin, Q1 RUM002N02T2L, Q2 RUM002N02T2L, U1 MB85RS2MTAPNF-G-BDERE1, U2 ATSAMD21G18A-A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

Commit message: udated by FZ
Parts:
- removed R16: 10K, Resistor_SMD:R_0402_1005Metric_Pad0.72x0.64mm_HandSolder
- Q1, Q2: value RUM002N02T2L -> PJE8408_R1_00001
Connections:
- U6 pad 3: /1V8_EN -> /VBAT
Routing:
- net /1V8_EN: track 8.94 -> 0.00 mm
- net /VBAT: track 41.8 -> 44.2 mm
Changed lines of the file:
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@@
       (net 1 "GND") (pinfunction "GND") (pintype "power_in"))
     (pad "3" smd roundrect (at -1.1375 0.95 270) (size 1.325 0.6) (layers "F.Cu" "F.Paste" "F.Mask") (roundrect_rratio 0.25)
-      (net 53 "/1V8_EN") (pinfunction "EN") (pintype "input"))
+      (net 4 "/VBAT") (pinfunction "EN") (pintype "input"))
     (pad "4" smd roundrect (at 1.1375 0.95 270) (size 1.325 0.6) (layers "F.Cu" "F.Paste" "F.Mask") (roundrect_rratio 0.25)
       (net 54 "unconnected-(U6-NC-Pad4)") (pinfunction "NC") (pintype "power_in+no_connect"))
@@
       (net 41 "/TXD") (pinfunction "PB23") (pintype "bidirectional"))
     (pad "39" smd roundrect (at 1.75 -4.1625) (size 0.3 1.475) (layers "F.Cu" "F.Paste" "F.Mask") (roundrect_rratio 0.25)
-      (net 53 "/1V8_EN") (pinfunction "PA27") (pintype "bidirectional"))
+      (net 53 "/1V8_EN") (pinfunction "PA27") (pintype "bidirectional+no_connect"))
     (pad "40" smd roundrect (at 1.25 -4.1625) (size 0.3 1.475) (layers "F.Cu" "F.Paste" "F.Mask") (roundrect_rratio 0.25)
       (net 17 "/~{RESET}") (pinfunction "~{RESET}") (pintype "input"))
     (pad "41" smd roundrect (at 0.75 -4.1625) (size 0.3 1.475) (layers "F.Cu" "F.Paste" "F.Mask") (roundrect_rratio 0.25)
-      (net 73 "/MPPT_EN") (pinfunction "PA28") (pintype "bidirectional+no_connect"))
+      (net 73 "/MPPT_EN") (pinfunction "PA28") (pintype "bidirectional"))
     (pad "42" smd roundrect (at 0.25 -4.1625) (size 0.3 1.475) (layers "F.Cu" "F.Paste" "F.Mask") (roundrect_rratio 0.25)
       (net 1 "GND") (pinfunction "GND") (pintype "passive"))
@@
         (effects (font (size 1.27 1.27) (thickness 0.254)))
     )
-    (fp_text value "RUM002N02T2L" (at 0 0 90) (layer "F.SilkS") hide
+    (fp_text value "PJE8408_R1_00001" (at 0 0 90) (layer "F.SilkS") hide
         (effects (font (size 1.27 1.27) (thickness 0.254)))
     )
@@
         (effects (font (size 1.27 1.27) (thickness 0.254)))
     )
-    (fp_text value "RUM002N02T2L" (at 0 0 90) (layer "F.SilkS") hide
+    (fp_text value "PJE8408_R1_00001" (at 0 0 90) (layer "F.SilkS") hide
         (effects (font (size 1.27 1.27) (thickness 0.254)))
     )
@@
     )
   )
-  (footprint "Resistor_SMD:R_0402_1005Metric_Pad0.72x0.64mm_HandSolder" (layer "F.Cu")
-    (at 147.18 90.708621 90)
-    (descr "Resistor SMD 0402 (1005 Metric), square (rectangular) end terminal, IPC_7351 nominal with elongated pad for handsoldering. (Body size source: IPC-SM-782 page 72, https://www.pcb-3d.com/wordpress/wp-content/uploads/ipc-sm-782a_amendment_1_and_2.pdf), generated with kicad-footprint-generator")
-    (tags "resistor handsolder")
-    (property "Sheetfile" "MCU.kicad_sch")
-    (property "Sheetname" "")
-    (property "ki_description" "Resistor, small symbol")
-    (property "ki_keywords" "R resistor")
-    (attr smd)
-    (fp_text reference "R16" (at 0 -1.17 90) (layer "F.SilkS") hide
-        (effects (font (size 1 1) (thickness 0.15)))
-    )
-    (fp_text value "10K" (at 0 1.17 90) (layer "F.Fab")
-        (effects (font (size 1 1) (thickness 0.15)))
-    )
-    (fp_text user "${REFERENCE}" (at 0 0 90) (layer "F.Fab")
-        (effects (font (size 0.26 0.26) (thickness 0.04)))
-    )
-    (fp_line (start -0.167621 -0.38) (end 0.167621 -0.38)
-      (stroke (width 0.12) (type solid)) (layer "F.SilkS"))
-    (fp_line (start -0.167621 0.38) (end 0.167621 0.38)
-      (stroke (width 0.12) (type solid)) (layer "F.SilkS"))
-    (fp_line (start -1.1 -0.47) (end 1.1 -0.47)
-      (stroke (width 0.05) (type solid)) (layer "F.CrtYd"))
-    (fp_line (start -1.1 0.47) (end -1.1 -0.47)
-      (stroke (width 0.05) (type solid)) (layer "F.CrtYd"))
-    (fp_line (start 1.1 -0.47) (end 1.1 0.47)
-      (stroke (width 0.05) (type solid)) (layer "F.CrtYd"))
-    (fp_line (start 1.1 0.47) (end -1.1 0.47)
-      (stroke (width 0.05) (type solid)) (layer "F.CrtYd"))
-    (fp_line (start -0.525 -0.27) (end 0.525 -0.27)
-      (stroke (width 0.1) (type solid)) (layer "F.Fab"))
-    (fp_line (start -0.525 0.27) (end -0.525 -0.27)
-      (stroke (width 0.1) (type solid)) (layer "F.Fab"))
-    (fp_line (start 0.525 -0.27) (end 0.525 0.27)
-      (stroke (width 0.1) (type solid)) (layer "F.Fab"))
-    (fp_line (start 0.525 0.27) (end -0.525 0.27)
-      (stroke (width 0.1) (type solid)) (layer "F.Fab"))
-    (pad "1" smd roundrect (at -0.5975 0 90) (size 0.715 0.64) (layers "F.Cu" "F.Paste" "F.Mask") (roundrect_rratio 0.25)
-      (net 53 "/1V8_EN") (pintype "passive"))
-    (pad "2" smd roundrect (at 0.5975 0 90) (size 0.715 0.64) (layers "F.Cu" "F.Paste" "F.Mask") (roundrect_rratio 0.25)
-      (net 1 "GND") (pintype "passive"))
-    (model "${KICAD6_3DMODEL_DIR}/Resistor_SMD.3dshapes/R_0402_1005Metric.wrl"
-      (offset (xyz 0 0 0))
-      (scale (xyz 1 1 1))
-      (rotate (xyz 0 0 0))
-    )
-  )
   (footprint "Connector_PinHeader_2.00mm:PinHeader_1x04_P2.00mm_Vertical" (layer "F.Cu")
     (at 168.51 97.10461)
@@
   (segment (start 166.3575 97.296121) (end 166.3575 96.268621) (width 0.1524) (layer "F.Cu") (net 3))
   (segment (start 166.3575 96.268621) (end 166.3275 96.238621) (width 0.1524) (layer "F.Cu") (net 3))
-  (segment (start 149.6025 88.188621) (end 145.094021 88.188621) (width 0.508) (layer "F.Cu") (net 4))
   (segment (start 142.75 91.568621) (end 143.69 91.568621) (width 0.1524) (layer "F.Cu") (net 4))
   (segment (start 150.4425 90.513621) (end 150.45 90.521121) (width 0.508) (layer "F.Cu") (net 4))
@@
   (segment (start 143.69 91.568621) (end 144.2675 90.991121) (width 0.1524) (layer "F.Cu") (net 4))
   (segment (start 134.3 102.008621) (end 133.66 101.368621) (width 0.1524) (layer "F.Cu") (net 4))
+  (segment (start 148.55 90.521121) (end 148.55 88.253621) (width 0.1524) (layer "F.Cu") (net 4))
   (segment (start 142.3675 90.521121) (end 142.3675 91.186121) (width 0.1524) (layer "F.Cu") (net 4))
   (segment (start 150.4425 89.028621) (end 149.6025 88.188621) (width 0.508) (layer "F.Cu") (net 4))
+  (segment (start 148.55 88.253621) (end 148.485 88.188621) (width 0.1524) (layer "F.Cu") (net 4))
   (segment (start 144.2675 90.521121) (end 144.2675 89.033621) (width 0.508) (layer "F.Cu") (net 4))
   (segment (start 144.2675 90.991121) (end 144.2675 90.521121) (width 0.1524) (layer "F.Cu") (net 4))
+  (segment (start 149.6025 88.188621) (end 148.485 88.188621) (width 0.508) (layer "F.Cu") (net 4))
   (segment (start 135.37 102.008621) (end 134.3 102.008621) (width 0.1524) (layer "F.Cu") (net 4))
   (segment (start 145.094021 87.74962) (end 143.81 86.465599) (width 0.508) (layer "F.Cu") (net 4))
@@
   (segment (start 144.2675 89.033621) (end 144.2625 89.028621) (width 0.508) (layer "F.Cu") (net 4))
   (segment (start 142.3675 91.186121) (end 142.75 91.568621) (width 0.1524) (layer "F.Cu") (net 4))
+  (segment (start 148.485 88.188621) (end 145.094021 88.188621) (width 0.508) (layer "F.Cu") (net 4))
   (segment (start 145.094021 88.188621) (end 144.2625 89.020142) (width 0.508) (layer "F.Cu") (net 4))
   (via (at 133.66 101.368621) (size 0.6604) (drill 0.3302) (layers "F.Cu" "B.Cu") (net 4))
@@
   (segment (start 156.04 97.150621) (end 156.748 97.858621) (width 0.1524) (layer "F.Cu") (net 52))
   (via (at 150.45 96.858621) (size 0.6604) (drill 0.3302) (layers "F.Cu" "B.Cu") (net 52))
-  (segment (start 147.18 94.348621) (end 147.18 93.958621) (width 0.1524) (layer "F.Cu") (net 53))
-  (segment (start 144.86 97.586121) (end 144.86 96.668621) (width 0.1524) (layer "F.Cu") (net 53))
-  (segment (start 147.18 91.306121) (end 147.765 91.306121) (width 0.1524) (layer "F.Cu") (net 53))
-  (segment (start 147.18 91.306121) (end 147.18 93.958621) (width 0.1524) (layer "F.Cu") (net 53))
-  (segment (start 147.765 91.306121) (end 148.55 90.521121) (width 0.1524) (layer "F.Cu") (net 53))
-  (segment (start 144.86 96.668621) (end 147.18 94.348621) (width 0.1524) (layer "F.Cu") (net 53))
   (segment (start 155.06 95.855529) (end 154.726908 96.188621) (width 0.1524) (layer "F.Cu") (net 69))
   (segment (start 152.65 96.188621) (end 152.63 96.208621) (width 0.1524) (layer "F.Cu") (net 69))
