File: PCB/MCU/MCU.kicad_sch (KiCad schematic)
At the start: 57 parts, among them IC2 LTC4311CSC6#TRPBF, J1 Conn_02x06_Odd_Even, J2 Conn_02x06_Odd_Even, J4 Conn_01x04_Pin, J5 RESET, J6 Conn_01x04_Pin, Q1 RUM002N02T2L, Q2 RUM002N02T2L, U1 MB85RS2MTAPNF-G-BDERE1, U2 ATSAMD21G18A-A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

Commit message: udated by FZ
Connections:
- net MPPT_EN: no longer J1.5 (Pin_5)
- new net VBUS: J1.5 (Pin_5)
- no-connect marks 9 -> 10
Other:
- moved on the sheet: J1, R20

Commit message: udated by FZ
Changed lines of the file:
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@@
     (effects (font (size 1.27 1.27)) (justify right bottom))
+  )
+  (label "LORA_FREQ_SELECT" (at 261.62 27.94 0) (fields_autoplaced)
+    (effects (font (size 1.27 1.27)) (justify left bottom))
   )
   (label "D12" (at 64.77 87.63 0) (fields_autoplaced)

Commit message: udated by FZ
Parts:
- Q1, Q2: value RUM002N02T2L -> PJE8408_R1_00001
Changed lines of the file:
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@@
       (effects (font (size 1.27 1.27)) (justify left))
     )
-    (property "Value" "RUM002N02T2L" (at 158.75 107.95 90)
+    (property "Value" "PJE8408_R1_00001" (at 158.75 107.95 90)
       (effects (font (size 1.27 1.27)) (justify left))
     )
@@
       (effects (font (size 1.27 1.27)) (justify left))
     )
-    (property "Value" "RUM002N02T2L" (at 168.91 93.98 90)
-      (effects (font (size 1.27 1.27)) (justify left))
-    )
+    (property "Value" "PJE8408_R1_00001" (at 168.91 93.98 90)
+      (effects (font (size 1.27 1.27)) (justify left))
+    )

Commit message: udated by FZ
Parts:
- removed R16: 10K, Resistor_SMD:R_0402_1005Metric_Pad0.72x0.64mm_HandSolder, symbol Device:R_Small
Connections:
- net 1V8_EN: no longer U6.3 (EN)
- net VBAT: now also U6.3 (EN)
Other:
- moved on the sheet: C2
Changed lines of the file:
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@@
   (junction (at 44.45 39.37) (diameter 0) (color 0 0 0 0)
   )
-  (junction (at 95.25 156.21) (diameter 0) (color 0 0 0 0)
-  )
   (junction (at 110.49 25.4) (diameter 0) (color 0 0 0 0)
   )
@@
   (junction (at 223.52 137.16) (diameter 0) (color 0 0 0 0)
   )
+  (junction (at 100.33 152.4) (diameter 0) (color 0 0 0 0)
+  )
   (junction (at 210.82 137.16) (diameter 0) (color 0 0 0 0)
   )
@@
   (junction (at 26.67 44.45) (diameter 0) (color 0 0 0 0)
   )
-  (junction (at 102.87 154.94) (diameter 0) (color 0 0 0 0)
-  )
   (junction (at 99.06 25.4) (diameter 0) (color 0 0 0 0)
   )
@@
   (junction (at 116.84 36.83) (diameter 0) (color 0 0 0 0)
   )
+  (no_connect (at 64.77 107.95))
   (no_connect (at 146.05 175.26))
   (no_connect (at 176.53 48.26))
@@
   (no_connect (at 73.66 46.99))
   (no_connect (at 146.05 38.1))
-  (no_connect (at 64.77 110.49))
   (no_connect (at 176.53 53.34))
   (no_connect (at 73.66 72.39))
@@
     (stroke (width 0) (type default))
   )
+  (wire (pts (xy 95.25 152.4) (xy 95.25 153.67))
+    (stroke (width 0) (type default))
+  )
   (wire (pts (xy 151.13 135.89) (xy 170.18 135.89))
     (stroke (width 0) (type default))
@@
     (stroke (width 0) (type default))
   )
-  (wire (pts (xy 102.87 158.75) (xy 102.87 154.94))
-    (stroke (width 0) (type default))
-  )
   (wire (pts (xy 91.44 129.54) (xy 91.44 130.81))
     (stroke (width 0) (type default))
@@
     (stroke (width 0) (type default))
   )
-  (wire (pts (xy 95.25 156.21) (xy 95.25 154.94))
-    (stroke (width 0) (type default))
-  )
   (wire (pts (xy 173.99 83.82) (xy 173.99 88.9))
     (stroke (width 0) (type default))
@@
     (stroke (width 0) (type default))
   )
-  (wire (pts (xy 109.22 59.69) (xy 115.57 59.69))
+  (wire (pts (xy 100.33 152.4) (xy 100.33 154.94))
     (stroke (width 0) (type default))
   )
-  (wire (pts (xy 195.58 40.64) (xy 204.47 40.64))
+  (wire (pts (xy 109.22 59.69) (xy 115.57 59.69))
     (stroke (width 0) (type default))
   )
-  (wire (pts (xy 100.33 152.4) (xy 100.33 149.86))
+  (wire (pts (xy 195.58 40.64) (xy 204.47 40.64))
     (stroke (width 0) (type default))
   )
@@
     (stroke (width 0) (type default))
   )
+  (wire (pts (xy 102.87 154.94) (xy 100.33 154.94))
+    (stroke (width 0) (type default))
+  )
   (wire (pts (xy 64.77 107.95) (xy 73.66 107.95))
     (stroke (width 0) (type default))
@@
     (stroke (width 0) (type default))
   )
-  (wire (pts (xy 97.79 158.75) (xy 97.79 156.21))
-    (stroke (width 0) (type default))
-  )
   (wire (pts (xy 69.85 160.02) (xy 69.85 161.29))
     (stroke (width 0) (type default))
@@
     (stroke (width 0) (type default))
   )
-  (wire (pts (xy 96.52 154.94) (xy 102.87 154.94))
-    (stroke (width 0) (type default))
-  )
   (wire (pts (xy 195.58 33.02) (xy 204.47 33.02))
     (stroke (width 0) (type default))
@@
     (stroke (width 0) (type default))
   )
-  (wire (pts (xy 97.79 156.21) (xy 95.25 156.21))
-    (stroke (width 0) (type default))
-  )
   (polyline (pts (xy 266.7 149.86) (xy 184.15 149.86))
     (stroke (width 0) (type default))
@@
     (stroke (width 0) (type default))
   )
+  (wire (pts (xy 95.25 160.02) (xy 95.25 158.75))
+    (stroke (width 0) (type default))
+  )
   (wire (pts (xy 116.84 25.4) (xy 116.84 27.94))
     (stroke (width 0) (type default))
@@
     (stroke (width 0) (type default))
   )
-  (wire (pts (xy 95.25 149.86) (xy 100.33 149.86))
+  (wire (pts (xy 95.25 152.4) (xy 100.33 152.4))
     (stroke (width 0) (type default))
   )
@@
     (effects (font (size 1.27 1.27)) (justify left bottom))
   )
-  (label "VBAT" (at 95.25 149.86 0) (fields_autoplaced)
+  (label "VBAT" (at 95.25 152.4 0) (fields_autoplaced)
     (effects (font (size 1.27 1.27)) (justify left bottom))
   )
@@
     (effects (font (size 1.27 1.27)) (justify right bottom))
   )
-  (label "1V8_EN" (at 96.52 154.94 0) (fields_autoplaced)
-    (effects (font (size 1.27 1.27)) (justify left bottom))
-  )
   (label "SDA" (at 257.175 129.54 180) (fields_autoplaced)
     (effects (font (size 1.27 1.27)) (justify right bottom))
@@
     )
   )
-  (symbol (lib_id "power:GND") (at 95.25 156.21 0) (unit 1)
+  (symbol (lib_id "power:GND") (at 95.25 160.02 0) (unit 1)
     (in_bom yes) (on_board yes) (dnp no) (fields_autoplaced)
-    (property "Reference" "#PWR05" (at 95.25 162.56 0)
+    (property "Reference" "#PWR05" (at 95.25 166.37 0)
       (effects (font (size 1.27 1.27)) hide)
     )
-    (property "Value" "GND" (at 95.25 160.7725 0)
+    (property "Value" "GND" (at 95.25 164.5825 0)
       (effects (font (size 1.27 1.27)))
     )
-    (property "Footprint" "" (at 95.25 156.21 0)
+    (property "Footprint" "" (at 95.25 160.02 0)
       (effects (font (size 1.27 1.27)) hide)
     )
-    (property "Datasheet" "" (at 95.25 156.21 0)
+    (property "Datasheet" "" (at 95.25 160.02 0)
       (effects (font (size 1.27 1.27)) hide)
     )
@@
     )
   )
-  (symbol (lib_id "Device:R_Small") (at 100.33 158.75 270) (unit 1)
-    (in_bom yes) (on_board yes) (dnp no)
-    (property "Reference" "R16" (at 100.33 160.528 90)
-      (effects (font (size 1.27 1.27)))
-    )
-    (property "Value" "10K" (at 100.33 156.718 90)
-      (effects (font (size 1.27 1.27)))
-    )
-    (property "Footprint" "Resistor_SMD:R_0402_1005Metric_Pad0.72x0.64mm_HandSolder" (at 100.33 158.75 0)
-      (effects (font (size 1.27 1.27)) hide)
-    )
-    (property "Datasheet" "~" (at 100.33 158.75 0)
-      (effects (font (size 1.27 1.27)) hide)
-    )
-    (pin "1")
-    (pin "2")
-    (instances
-      (project "MCU"
-        (path "/e63e39d7-6ac0-4ffd-8aa3-1841a4541b55"
-          (reference "R16") (unit 1)
-        )
-      )
-    )
-  )
   (symbol (lib_id "Device:C_Small") (at 30.48 39.37 90) (unit 1)
     (in_bom yes) (on_board yes) (dnp no)
@@
     )
   )
-  (symbol (lib_id "Device:C_Small") (at 95.25 152.4 0) (unit 1)
+  (symbol (lib_id "Device:C_Small") (at 95.25 156.21 0) (unit 1)
     (in_bom yes) (on_board yes) (dnp no)
-    (property "Reference" "C2" (at 90.17 151.13 0)
+    (property "Reference" "C2" (at 90.17 154.94 0)
       (effects (font (size 1.27 1.27)) (justify left))
     )
-    (property "Value" "0.1uF" (at 89.408 154.94 0)
+    (property "Value" "0.1uF" (at 89.408 158.75 0)
       (effects (font (size 1.27 1.27)) (justify left))
     )
-    (property "Footprint" "Capacitor_SMD:C_0402_1005Metric_Pad0.74x0.62mm_HandSolder" (at 95.25 152.4 0)
+    (property "Footprint" "Capacitor_SMD:C_0402_1005Metric_Pad0.74x0.62mm_HandSolder" (at 95.25 156.21 0)
       (effects (font (size 1.27 1.27)) hide)
     )
-    (property "Datasheet" "~" (at 95.25 152.4 0)
+    (property "Datasheet" "~" (at 95.25 156.21 0)
       (effects (font (size 1.27 1.27)) hide)
     )

Commit message: udated by FZ
Other:
- note added: "Switch these 2 pins"
Changed lines of the file:
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@@
     (stroke (width 0) (type default))
+  )
+  (rectangle (start 108.204 99.06) (end 128.27 102.108)
+    (stroke (width 0) (type default))
+    (fill (type none))
   )
   (text "ICM-20948" (at 133.35 20.32 0)
@@
     (effects (font (size 2.54 2.54) (thickness 0.508) bold) (justify left bottom))
   )
+  (text "Switch these 2 pins" (at 108.458 101.6 0)
+    (effects (font (size 1.27 1.27)) (justify left bottom))
+  )
   (text "SSQ-106-23-G-D" (at 216.916 20.32 0)

Commit message: auto stand work
Connections:
- net 1V8_EN: now also U6.3 (EN)
- net VBAT: no longer U6.3 (EN)
- no-connect marks 10 -> 9
Changed lines of the file:
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@@
   (junction (at 223.52 137.16) (diameter 0) (color 0 0 0 0)
   )
-  (junction (at 100.33 152.4) (diameter 0) (color 0 0 0 0)
-  )
   (junction (at 210.82 137.16) (diameter 0) (color 0 0 0 0)
   )
@@
   (junction (at 116.84 36.83) (diameter 0) (color 0 0 0 0)
   )
-  (no_connect (at 64.77 107.95))
   (no_connect (at 146.05 175.26))
   (no_connect (at 176.53 48.26))
@@
     (stroke (width 0) (type default))
   )
-  (wire (pts (xy 100.33 152.4) (xy 100.33 154.94))
-    (stroke (width 0) (type default))
-  )
   (wire (pts (xy 109.22 59.69) (xy 115.57 59.69))
     (stroke (width 0) (type default))
@@
     (stroke (width 0) (type default))
   )
-  (wire (pts (xy 102.87 154.94) (xy 100.33 154.94))
+  (wire (pts (xy 102.87 154.94) (xy 96.52 154.94))
     (stroke (width 0) (type default))
   )
@@
     (stroke (width 0) (type default))
   )
-  (wire (pts (xy 100.33 152.4) (xy 102.87 152.4))
+  (wire (pts (xy 95.25 152.4) (xy 102.87 152.4))
     (stroke (width 0) (type default))
   )
@@
   )
   (wire (pts (xy 210.82 129.54) (xy 224.79 129.54))
-    (stroke (width 0) (type default))
-  )
-  (wire (pts (xy 95.25 152.4) (xy 100.33 152.4))
     (stroke (width 0) (type default))
   )
@@
     (effects (font (size 1.27 1.27)) (justify right bottom))
   )
+  (label "1V8_EN" (at 96.52 154.94 0) (fields_autoplaced)
+    (effects (font (size 1.27 1.27)) (justify left bottom))
+  )
   (label "A5" (at 115.57 44.45 180) (fields_autoplaced)
