File: PCB/PWR/V2/PWR.kicad_pcb (KiCad board)
At the start: 2 copper layers, 40 x 46.2 mm, 39 parts, among them J1 Switch conn, J2 Conn_02x06_Odd_Even, J3 Battery, J4 Solar cell, U1 AP2112K-3.3, U2 BQ25570, U3 AP2112K-1.8, U4 MCP73831-2-OT

Commit message: udated by FZ
Parts:
- removed C10, C12: 47uF, LED_SMD:LED_0805_2012Metric_Pad1.15x1.40mm_HandSolder
- removed C11, C9: 0.1uF, Capacitor_SMD:C_0402_1005Metric_Pad0.74x0.62mm_HandSolder
- removed TP1, TP2, TP3, TP4: TestPoint_Alt, TestPoint:TestPoint_Pad_1.0x1.0mm
- removed U1: AP2112K-3.3, Package_TO_SOT_SMD:SOT-23-5
- removed U3: AP2112K-1.8, Package_TO_SOT_SMD:SOT-23-5
- added J10: Battery, Connector_Molex:Molex_Micro-Latch_53253-0270_1x02_P2.00mm_Vertical, F.Cu at (132.2, 96.4)
- added J5: Conn_02x06_Odd_Even, Connector_PinHeader_2.54mm:PinHeader_2x06_P2.54mm_Vertical, F.Cu at (140.7, 81.8)
- added J6: Conn_02x06_Odd_Even, Connector_PinHeader_2.54mm:PinHeader_2x06_P2.54mm_Vertical, F.Cu at (153.3, 109.0)
- added J7: Battery, Connector_Molex:Molex_Micro-Latch_53253-0270_1x02_P2.00mm_Vertical, F.Cu at (158.8, 81.6)
- added J8: Battery, Connector_Molex:Molex_Micro-Latch_53253-0270_1x02_P2.00mm_Vertical, F.Cu at (161.8, 94.4)
- added J9: Battery, Connector_Molex:Molex_Micro-Latch_53253-0270_1x02_P2.00mm_Vertical, F.Cu at (133.4, 82.6)
- added R2: NC, Resistor_SMD:R_0603_1608Metric_Pad0.98x0.95mm_HandSolder, B.Cu at (145.8, 86.1)
- C5: footprint Capacitor_SMD:C_1206_3216Metric_Pad1.33x1.80mm_HandSolder -> Capacitor_SMD:C_0603_1608Metric_Pad1.08x0.95mm_HandSolder
- J1: value Switch conn -> Battery; footprint Connector_PinHeader_2.54mm:PinHeader_1x02_P2.54mm_Vertical -> Connector_Molex:Molex_Micro-Latch_53253-0270_1x02_P2.00mm_Vertical
- J2: value Conn_02x06_Odd_Even -> Battery; footprint Connector_PinHeader_2.54mm:PinHeader_2x06_P2.54mm_Vertical -> Connector_PinHeader_2.00mm:PinHeader_2x01_P2.00mm_Vertical
- J4: value Solar cell -> Battery; footprint Connector_PinHeader_2.00mm:PinHeader_2x01_P2.00mm_Vertical -> Connector_Molex:Molex_Micro-Latch_53253-0270_1x02_P2.00mm_Vertical
- R1: footprint Resistor_SMD:R_1206_3216Metric_Pad1.30x1.75mm_HandSolder -> Resistor_SMD:R_0603_1608Metric_Pad0.98x0.95mm_HandSolder
- moved J3 36.8 mm to (128.5, 94.6), turned to -90 degrees
- moved R1 23.9 mm to (143.1, 86.0), turned to 180 degrees
- moved C5 23.2 mm to (143.1, 84.5), turned to 0 degrees
- moved J1 21.9 mm to (135.2, 109.2), turned to 150 degrees
- moved J4 17.1 mm to (160.6, 108.2), turned to -150 degrees
- moved R15 11.6 mm to (157.8, 89.8), turned to -90 degrees
- moved D1 11.0 mm to (154.7, 89.1)
- moved C4 9.73 mm to (153.7, 93.4)
- moved U4 9.62 mm to (156.7, 93.3)
- moved C6 9.54 mm to (153.2, 103.0)
- moved L1 9.09 mm to (150.0, 103.0)
- moved R16 8.99 mm to (154.6, 90.7)
- moved L2 8.49 mm to (149.9, 92.1)
- moved C7 8.25 mm to (145.6, 90.2)
- moved C8 8.25 mm to (137.4, 92.2)
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Connections:
- J1 pad 1: unconnected-(J1-Pin_1-Pad1) -> /SC
- J1 pad 2: /VBAT -> GND
- J2 pad 1: GND -> /VBAT
- J2 pad 2: /~{EN} -> /BATTERY
- J4 pad 2: /SC -> GND
- R13 pad 2: /~{EN} -> /D8
- U2 pad 13: /VBAT_OK -> /VBAT_OK_t
- U2 pad 5: /~{EN} -> /D8
Routing:
- net /SC: track 29.8 -> 104.9 mm
- net /VBAT_OK: track 24.1 -> 0.00 mm, vias 1 -> 0
- net /~{EN}: track 23.6 -> 0.00 mm, vias 2 -> 0
- net /D8: track 0.00 -> 20.0 mm, vias 0 -> 2
- net /VBAT: track 75.7 -> 56.0 mm, vias 4 -> 2
- net /VBAT_OK_t: track 0.00 -> 19.5 mm, vias 0 -> 1
- net +1V8: track 13.8 -> 0.00 mm
- net +3V3: track 11.0 -> 0.00 mm
- net +5V: track 38.1 -> 30.6 mm, vias 3 -> 1
- net /A3: track 0.00 -> 6.99 mm
- net Net-(D1-K): track 4.90 -> 1.66 mm
- net /BATTERY: track 0.00 -> 3.09 mm
- net Net-(U2-VOUT): track 14.8 -> 12.7 mm
- net Net-(U4-STAT): track 2.80 -> 1.66 mm
- net GND: vias 93 -> 50
Other:
- outline, holes or cut-outs redrawn
- board text removed: "HEXSENSE SVALBARD PWR_V1 FANGZHENG LIU MIT MEDIA LAB ResEnv"
