File: PCB/PWR/V2/PWR.kicad_sch (KiCad schematic)
At the start: 39 parts, among them J1 Switch conn, J2 Conn_02x06_Odd_Even, J3 Battery, J4 Solar cell, U1 AP2112K-3.3, U2 BQ25570, U3 AP2112K-1.8, U4 MCP73831-2-OT

Commit message: udated by FZ
Parts:
- removed C10, C12: 47uF, LED_SMD:LED_0805_2012Metric_Pad1.15x1.40mm_HandSolder, symbol Device:C_Polarized_Small_US
- removed C11, C9: 0.1uF, Capacitor_SMD:C_0402_1005Metric_Pad0.74x0.62mm_HandSolder, symbol Device:C_Small
- removed J1: Switch conn, Connector_PinHeader_2.54mm:PinHeader_1x02_P2.54mm_Vertical, symbol Connector:Conn_01x02_Pin
- removed J2: Conn_02x06_Odd_Even, Connector_PinHeader_2.54mm:PinHeader_2x06_P2.54mm_Vertical, symbol Connector_Generic:Conn_02x06_Odd_Even
- removed TP1, TP2, TP3, TP4: TestPoint_Alt, TestPoint:TestPoint_Pad_1.0x1.0mm, symbol Connector:TestPoint_Alt
- removed U1: AP2112K-3.3, Package_TO_SOT_SMD:SOT-23-5, symbol Regulator_Linear:AP2112K-3.3
- removed U3: AP2112K-1.8, Package_TO_SOT_SMD:SOT-23-5, symbol Regulator_Linear:AP2112K-1.8
- added J1, J10, J7, J8, J9: Battery, Connector_Molex:Molex_Micro-Latch_53253-0270_1x02_P2.00mm_Vertical, symbol Connector:Conn_01x02_Male
- added J2: Battery, Connector_PinHeader_2.00mm:PinHeader_2x01_P2.00mm_Vertical, symbol Connector:Conn_01x02_Male
- added J5, J6: Conn_02x06_Odd_Even, Connector_PinHeader_2.54mm:PinHeader_2x06_P2.54mm_Vertical, symbol Connector_Generic:Conn_02x06_Odd_Even
- added R2: NC, Resistor_SMD:R_0603_1608Metric_Pad0.98x0.95mm_HandSolder, symbol Device:R_Small
- C5: footprint Capacitor_SMD:C_1206_3216Metric_Pad1.33x1.80mm_HandSolder -> Capacitor_SMD:C_0603_1608Metric_Pad1.08x0.95mm_HandSolder
- J4: value Solar cell -> Battery; footprint Connector_PinHeader_2.00mm:PinHeader_2x01_P2.00mm_Vertical -> Connector_Molex:Molex_Micro-Latch_53253-0270_1x02_P2.00mm_Vertical
- R1: footprint Resistor_SMD:R_1206_3216Metric_Pad1.30x1.75mm_HandSolder -> Resistor_SMD:R_0603_1608Metric_Pad0.98x0.95mm_HandSolder
Connections:
- net +5V: now also J5.5 (Pin_5)
- net BATTERY: now also J2.2 (Pin_2)
- net GND: now also J4.2 (Pin_2), J1.2 (Pin_2), J10.2 (Pin_2), J5.10 (Pin_10), J5.8 (Pin_8), J6.10 (Pin_10), J6.12 (Pin_12), J7.2 (Pin_2), J8.2 (Pin_2), J9.2 (Pin_2)
- net SC: now also J1.1 (Pin_1), J10.1 (Pin_1), J7.1 (Pin_1), J8.1 (Pin_1), J9.1 (Pin_1); no longer J4.2 (Pin_2)
- net VBAT: now also J2.1 (Pin_1), J5.1 (Pin_1)
- net VBAT_OK renamed VBAT_OK_t
- net VBAT_OK_t: now also R2.2
- net ~{EN} renamed D8
- net D8: now also J5.2 (Pin_2)
- new net A2: J5.6 (Pin_6)
- new net A3: J5.4 (Pin_4), R2.1
- new net A4: J6.8 (Pin_8)
- new net A5: J5.3 (Pin_3)
- new net D1: J6.4 (Pin_4)
- new net D10: J6.2 (Pin_2)
- new net D12: J6.1 (Pin_1)
- new net D2: J6.7 (Pin_7)
- new net D3: J6.6 (Pin_6)
- new net D4: J6.11 (Pin_11)
- new net MISO: J6.9 (Pin_9)
- new net MOSI: J6.3 (Pin_3)
- new net RXD: J5.7 (Pin_7)
- new net SCK: J6.5 (Pin_5)
- new net SCL: J5.12 (Pin_12)
- new net SDA: J5.11 (Pin_11)
- new net TXD: J5.9 (Pin_9)
- no-connect marks 1 -> 0
Other:
- note removed: "Power supply"
- moved on the sheet: C2, C3, C4, J3
