File: PCB/SIDE/V1/SIDE.kicad_pcb (KiCad board)
At the start: 2 copper layers, 29 x 109 mm, 21 parts, among them IC1 VEML6030-GS15, J1 pin, J2 pin, J4 SM06B-SRSS-TB(LF)(SN), Q1 PJE8408_R1_00001, Q2 PJE8408_R1_00001, U1 AS7341DLG, U2 TMP112xxDRL, U3 SHT4x

Commit message: udated by FZ
Parts:
- removed C1, C2: 0.1uF, Capacitor_SMD:C_0603_1608Metric_Pad1.08x0.95mm_HandSolder
- removed IC1: VEML6030-GS15, SamacSys_Parts:VEML6030GS15
- removed J4: SM06B-SRSS-TB(LF)(SN), Connector_JST:JST_SH_SM06B-SRSS-TB_1x06-1MP_P1.00mm_Horizontal
- removed Q1, Q2: PJE8408_R1_00001, SamacSys_Parts:SOTFL50P160X60-3N
- removed R1, R11, R2, R3, R4, R5: 4.7k, Resistor_SMD:R_0603_1608Metric_Pad0.98x0.95mm_HandSolder
- removed SC1: Solar_Cell, Mylib:KXOB201K04F-TR
- removed U1: AS7341DLG, Package_LGA:AMS_OLGA-8_2x3.1mm_P0.8mm
- removed U2: TMP112xxDRL, Package_TO_SOT_SMD:SOT-563
- removed U3: SHT4x, Sensor_Humidity:Sensirion_DFN-4_1.5x1.5mm_P0.8mm_SHT4x_NoCentralPad
- added J3: SM02B-SRSS-TB_LFSN_, SamacSys_Parts:SM02B-SRSS-TB, B.Cu at (182.3, 121.4)
- moved D1 78.4 mm to (189.4, 123.0), turned to -90 degrees
- moved J1 39.4 mm to (179.8, 79.9)
- moved J2 39.4 mm to (179.8, 75.6)
- moved R6 37.8 mm to (172.3, 83.9)
- moved SC2 36.2 mm to (186.7, 116.0)
Connections:
- SC2 pad 1: Net-(SC1--) -> Net-(D1-A)
Routing:
- net Net-(SC1--): track 54.0 -> 0.00 mm, vias 19 -> 0
- net /SCL: track 52.9 -> 0.00 mm, vias 1 -> 0
- net +3V3: track 46.8 -> 0.00 mm, vias 5 -> 0
- net /SDA: track 43.2 -> 0.00 mm, vias 1 -> 0
- net +1V8: track 42.9 -> 0.00 mm, vias 3 -> 0
- net /SC: track 19.6 -> 7.95 mm
- net Net-(D1-A): track 0.00 -> 6.11 mm, vias 13 -> 4
- net Net-(IC1-ADDR): track 5.35 -> 0.00 mm, vias 1 -> 0
- net GND: track 4.77 -> 0.00 mm, vias 62 -> 106
- net /SCL_1.8: track 3.98 -> 0.00 mm, vias 1 -> 0
- net /SDA_1.8: track 2.78 -> 0.00 mm, vias 1 -> 0
- net /BR+: track 10.7 -> 8.29 mm
- net Net-(U2-ADD0): track 1.47 -> 0.00 mm
- net /BR-: track 8.26 -> 9.14 mm
- removed copper zone on B.Cu, net Net-(D1-A)
- removed copper zone on B.Cu, net Net-(SC1--)
Other:
- board size 29 x 109 mm -> 29 x 68 mm
- board text added: "MIT Media Lab - ResEnv HexSense - Canary Islands"
- board text removed: "MIT Media Lab - Responsive Environments HexSense - Svalbard Mission"
