File: PCB/SIDE/V1/SIDE.kicad_sch (KiCad schematic)
At the start: 21 parts, among them IC1 VEML6030-GS15, J1 pin, J2 pin, J4 SM06B-SRSS-TB(LF)(SN), Q1 PJE8408_R1_00001, Q2 PJE8408_R1_00001, U1 AS7341DLG, U2 TMP112xxDRL, U3 SHT4x

Commit message: udated by FZ
Parts:
- removed C1, C2: 0.1uF, Capacitor_SMD:C_0603_1608Metric_Pad1.08x0.95mm_HandSolder, symbol Device:C_Small
- removed IC1: VEML6030-GS15, SamacSys_Parts:VEML6030GS15, symbol SamacSys_Parts:VEML6030-GS15
- removed J4: SM06B-SRSS-TB(LF)(SN), Connector_JST:JST_SH_SM06B-SRSS-TB_1x06-1MP_P1.00mm_Horizontal, symbol Mylib:BM06B-SURS-TF(LF)(SN)
- removed Q1, Q2: PJE8408_R1_00001, SamacSys_Parts:SOTFL50P160X60-3N, symbol SamacSys_Parts:PJE8408_R1_00001
- removed R1, R11, R2, R3, R4, R5: 4.7k, Resistor_SMD:R_0603_1608Metric_Pad0.98x0.95mm_HandSolder, symbol Device:R_Small
- removed SC1: Solar_Cell, Mylib:KXOB201K04F-TR, symbol Device:Solar_Cell
- removed U1: AS7341DLG, Package_LGA:AMS_OLGA-8_2x3.1mm_P0.8mm, symbol Sensor_Optical:AS7341DLG
- removed U2: TMP112xxDRL, Package_TO_SOT_SMD:SOT-563, symbol Sensor_Temperature:TMP112xxDRL
- removed U3: SHT4x, Sensor_Humidity:Sensirion_DFN-4_1.5x1.5mm_P0.8mm_SHT4x_NoCentralPad, symbol Sensor_Humidity:SHT4x
- added J3: SM02B-SRSS-TB_LFSN_, SM02B-SRSS-TB, symbol SamacSys_Parts:SM02B-SRSS-TB_LFSN_
Connections:
- net GND: now also J3.2
- net SC: now also J3.1
- net at SC2.1 (+): now also D1.2 (A)
- no-connect marks 5 -> 0
Other:
- note added: "CUS08F30,H3F"
- note removed: "AS7341 Spectro"
- note removed: "Ambient light sensor"
- note removed: "SHT4x"
- note removed: "TMP112 - Body temperature"
- moved on the sheet: D1, J1, J2, R6, SC2

Commit message: udated by FZ
Parts:
- J3: footprint SM02B-SRSS-TB -> SamacSys_Parts:SM02B-SRSS-TB
Connections:
- net GND: now also J3.3, J3.4
Changed lines of the file:
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@@
     (comment 1 "Fangzheng Liu")
   )
+  (junction (at 55.88 71.12) (diameter 0) (color 0 0 0 0)
+  )
+  (junction (at 64.77 71.12) (diameter 0) (color 0 0 0 0)
+  )
+  (wire (pts (xy 55.88 71.12) (xy 64.77 71.12))
+    (stroke (width 0) (type default))
+  )
   (polyline (pts (xy 39.37 13.97) (xy 39.37 49.53))
     (stroke (width 0) (type default))
@@
     (stroke (width 0) (type default))
   )
+  (wire (pts (xy 64.77 71.12) (xy 64.77 63.5))
+    (stroke (width 0) (type default))
+  )
+  (wire (pts (xy 64.77 72.39) (xy 64.77 71.12))
+    (stroke (width 0) (type default))
+  )
   (polyline (pts (xy 38.1 49.53) (xy 13.97 49.53))
     (stroke (width 0) (type default))
   )
-  (wire (pts (xy 41.91 67.31) (xy 44.45 67.31))
+  (wire (pts (xy 41.91 63.5) (xy 44.45 63.5))
+    (stroke (width 0) (type default))
+  )
+  (wire (pts (xy 53.34 71.12) (xy 55.88 71.12))
     (stroke (width 0) (type default))
   )
@@
     (effects (font (size 1.27 1.27)) (justify left bottom))
   )
-  (label "SC" (at 41.91 67.31 0) (fields_autoplaced)
+  (label "SC" (at 41.91 63.5 0) (fields_autoplaced)
     (effects (font (size 1.27 1.27)) (justify left bottom))
   )
@@
     )
   )
-  (symbol (lib_id "SamacSys_Parts:SM02B-SRSS-TB_LFSN_") (at 44.45 67.31 0) (unit 1)
-    (in_bom yes) (on_board yes) (dnp no) (fields_autoplaced)
-    (property "Reference" "J3" (at 54.61 61.2408 0)
-      (effects (font (size 1.27 1.27)))
-    )
-    (property "Value" "SM02B-SRSS-TB_LFSN_" (at 54.61 63.2888 0)
-      (effects (font (size 1.27 1.27)))
-    )
-    (property "Footprint" "SM02B-SRSS-TB" (at 60.96 64.77 0)
-      (effects (font (size 1.27 1.27)) (justify left) hide)
-    )
-    (property "Datasheet" "" (at 60.96 67.31 0)
-      (effects (font (size 1.27 1.27)) (justify left) hide)
-    )
-    (property "Description" "2 way side entry SMT header,1mm pitch JST SH Series, 1mm Pitch 2 Way 1 Row Shrouded Right Angle PCB Header, Surface Mount, Solder Termination" (at 60.96 69.85 0)
-      (effects (font (size 1.27 1.27)) (justify left) hide)
-    )
-    (property "Height" "" (at 60.96 72.39 0)
-      (effects (font (size 1.27 1.27)) (justify left) hide)
-    )
-    (property "Manufacturer_Name" "JST (JAPAN SOLDERLESS TERMINALS)" (at 60.96 74.93 0)
-      (effects (font (size 1.27 1.27)) (justify left) hide)
-    )
-    (property "Manufacturer_Part_Number" "SM02B-SRSS-TB(LFSN)" (at 60.96 77.47 0)
-      (effects (font (size 1.27 1.27)) (justify left) hide)
-    )
-    (property "Mouser Part Number" "" (at 60.96 80.01 0)
-      (effects (font (size 1.27 1.27)) (justify left) hide)
-    )
-    (property "Mouser Price/Stock" "" (at 60.96 82.55 0)
-      (effects (font (size 1.27 1.27)) (justify left) hide)
-    )
-    (property "Arrow Part Number" "" (at 60.96 85.09 0)
-      (effects (font (size 1.27 1.27)) (justify left) hide)
-    )
-    (property "Arrow Price/Stock" "" (at 60.96 87.63 0)
+  (symbol (lib_id "SamacSys_Parts:SM02B-SRSS-TB_LFSN_") (at 44.45 63.5 0) (unit 1)
+    (in_bom yes) (on_board yes) (dnp no) (fields_autoplaced)
+    (property "Reference" "J3" (at 54.61 57.4308 0)
+      (effects (font (size 1.27 1.27)))
+    )
+    (property "Value" "SM02B-SRSS-TB_LFSN_" (at 54.61 59.4788 0)
+      (effects (font (size 1.27 1.27)))
+    )
+    (property "Footprint" "SamacSys_Parts:SM02B-SRSS-TB" (at 60.96 60.96 0)
+      (effects (font (size 1.27 1.27)) (justify left) hide)
+    )
+    (property "Datasheet" "" (at 60.96 63.5 0)
+      (effects (font (size 1.27 1.27)) (justify left) hide)
+    )
+    (property "Description" "2 way side entry SMT header,1mm pitch JST SH Series, 1mm Pitch 2 Way 1 Row Shrouded Right Angle PCB Header, Surface Mount, Solder Termination" (at 60.96 66.04 0)
+      (effects (font (size 1.27 1.27)) (justify left) hide)
+    )
+    (property "Height" "" (at 60.96 68.58 0)
+      (effects (font (size 1.27 1.27)) (justify left) hide)
+    )
+    (property "Manufacturer_Name" "JST (JAPAN SOLDERLESS TERMINALS)" (at 60.96 71.12 0)
+      (effects (font (size 1.27 1.27)) (justify left) hide)
+    )
+    (property "Manufacturer_Part_Number" "SM02B-SRSS-TB(LFSN)" (at 60.96 73.66 0)
+      (effects (font (size 1.27 1.27)) (justify left) hide)
+    )
+    (property "Mouser Part Number" "" (at 60.96 76.2 0)
+      (effects (font (size 1.27 1.27)) (justify left) hide)
+    )
+    (property "Mouser Price/Stock" "" (at 60.96 78.74 0)
+      (effects (font (size 1.27 1.27)) (justify left) hide)
+    )
+    (property "Arrow Part Number" "" (at 60.96 81.28 0)
+      (effects (font (size 1.27 1.27)) (justify left) hide)
+    )
+    (property "Arrow Price/Stock" "" (at 60.96 83.82 0)
       (effects (font (size 1.27 1.27)) (justify left) hide)
     )
     (pin "1")
     (pin "2")
+    (pin "3")
+    (pin "4")
     (instances
       (project "SIDE"
@@
     )
   )
-  (symbol (lib_id "power:GND") (at 64.77 67.31 0) (unit 1)
-    (in_bom yes) (on_board yes) (dnp no) (fields_autoplaced)
-    (property "Reference" "#PWR0119" (at 64.77 73.66 0)
-      (effects (font (size 1.27 1.27)) hide)
-    )
-    (property "Value" "GND" (at 64.77 71.7534 0)
-      (effects (font (size 1.27 1.27)))
-    )
-    (property "Footprint" "" (at 64.77 67.31 0)
-      (effects (font (size 1.27 1.27)) hide)
-    )
-    (property "Datasheet" "" (at 64.77 67.31 0)
-      (effects (font (size 1.27 1.27)) hide)
-    )
+  (symbol (lib_id "power:GND") (at 64.77 72.39 0) (unit 1)
+    (in_bom yes) (on_board yes) (dnp no) (fields_autoplaced)
+    (property "Reference" "#PWR0119" (at 64.77 78.74 0)
+      (effects (font (size 1.27 1.27)) hide)
+    )
+    (property "Value" "GND" (at 64.77 76.8334 0)
+      (effects (font (size 1.27 1.27)))
+    )
+    (property "Footprint" "" (at 64.77 72.39 0)
+      (effects (font (size 1.27 1.27)) hide)
+    )
+    (property "Datasheet" "" (at 64.77 72.39 0)
+      (effects (font (size 1.27 1.27)) hide)
+    )
