File: PCB/CAMERA_ADAPTER/CAMERA_ADAPTER.kicad_sch (KiCad schematic)
At the start: 12 parts, among them J1 Conn_02x06_Odd_Even, J10 Switch, J2 Conn_02x06_Odd_Even, J3 Conn_02x06_Odd_Even

Commit message: udated by FZ
Parts:
- removed D1, D2: LED, LED_SMD:LED_1206_3216Metric_Pad1.42x1.75mm_HandSolder, symbol Device:LED
- removed J10: Switch, Connector_PinHeader_2.00mm:PinHeader_1x02_P2.00mm_Vertical, symbol Connector:Conn_01x02_Pin
- removed J3: Conn_02x06_Odd_Even, Connector_PinHeader_2.54mm:PinHeader_2x06_P2.54mm_Vertical, symbol Connector_Generic:Conn_02x06_Odd_Even
- removed R1: 1M, Resistor_SMD:R_0603_1608Metric_Pad0.98x0.95mm_HandSolder, symbol Device:R_Small
- removed S1: 500SSP1S2M2QEA, Mylib:SW_500SSP1S2M2QEA, symbol 500SSP1S2M2QEA:500SSP1S2M2QEA
- removed TP1, TP2, TP3, TP4: TestPoint, TestPoint:TestPoint_Pad_1.0x1.0mm, symbol Connector:TestPoint
- added C13, C2: 0.1uF, Capacitor_SMD:C_0603_1608Metric_Pad1.08x0.95mm_HandSolder, symbol Device:C_Small
- added C3, C4, C5, C6, C7, C8, C9: 0.1uF, Capacitor_SMD:C_0402_1005Metric_Pad0.74x0.62mm_HandSolder, symbol Device:C_Small
- added D1: RED, LED_SMD:LED_0603_1608Metric_Pad1.05x0.95mm_HandSolder, symbol Device:LED_Small_Filled
- added J3, J4, J5, J6, J7, J8: BM06B-SRSS-TBT(LF)(SN), Connector_JST:JST_SH_BM06B-SRSS-TB_1x06-1MP_P1.00mm_Vertical, symbol Mylib:BM06B-SURS-TF(LF)(SN)
- added J9: Battery, Connector_PinHeader_2.00mm:PinHeader_1x02_P2.00mm_Vertical, symbol Connector:Conn_01x02_Pin
- added R10, R11, R5, R6, R7, R8, R9: 10k, Resistor_SMD:R_0402_1005Metric_Pad0.72x0.64mm_HandSolder, symbol Device:R_Small
- added R15, R16: 1k, Resistor_SMD:R_0603_1608Metric_Pad0.98x0.95mm_HandSolder, symbol Device:R_Small
- added R3, R4: NC, Resistor_SMD:R_0603_1608Metric_Pad0.98x0.95mm_HandSolder, symbol Device:R_Small
- added U2: TCA9534, Package_SO:TSSOP-16_4.4x5mm_P0.65mm, symbol Interface_Expansion:TCA9534
- added U3, U4, U5, U6, U7, U8, U9: AP2112K-3.3, Package_TO_SOT_SMD:SOT-23-5, symbol Regulator_Linear:AP2112K-3.3
- added U4: MCP73831-2-OT, Package_TO_SOT_SMD:SOT-23-5, symbol Battery_Management:MCP73831-2-OT
Connections:
- net +5V: now also C13.1, D1.2 (A), U4.4 (VDD)
- net A2: now also J3.5
- net A4: now also R11.1, U9.3 (EN)
- net A5: now also J4.5
- net D1: now also J7.5
- net D12: now also J5.5
- net D2: now also J6.5
- net D3: now also J8.5
- net GND: now also C13.2, C2.2, C3.2, C4.2, C5.2, C6.2, C7.2, C8.2, C9.2, J3.6, J3.MP, J4.6, J4.MP, J5.6, J5.MP, J6.6, J6.MP, J7.6, J7.MP, J8.6, J8.MP, J9.1 (Pin_1), R10.2, R11.2, R15.1, R5.2, R6.2, R7.2, R8.2, R9.2, U2.1 (A0), U2.2 (A1), U2.3 (A2), U2.8 (GND), U3.2 (GND), U4.2 (GND), U4.2 (VSS), U5.2 (GND), U6.2 (GND), U7.2 (GND), U8.2 (GND), U9.2 (GND)
- net MISO: now also J3.2, J4.2, J5.2, J6.2, J7.2, J8.2
- net MOSI: now also J3.4, J4.4, J5.4, J6.4, J7.4, J8.4
- net SCK: now also J3.3, J4.3, J5.3, J6.3, J7.3, J8.3
- net SCL: now also R4.2, U2.14 (SCL)
- net SDA: now also R3.2, U2.15 (SDA)
- new net: R16.1, U4.1 (STAT)
- new net: D1.1 (K), R16.2
- new net: R15.2, U4.5 (PROG)
- new net CAM_BAT: C3.1, C4.1, C5.1, C6.1, C7.1, C8.1, C9.1, J9.2 (Pin_2), U3.1 (VIN), U4.1 (VIN), U4.3 (VBAT), U5.1 (VIN), U6.1 (VIN), U7.1 (VIN), U8.1 (VIN), U9.1 (VIN)
- new net EN_1: R5.1, U2.11 (P6), U3.3 (EN)
- new net EN_2: R9.1, U2.10 (P5), U4.3 (EN)
- new net EN_3: R8.1, U2.9 (P4), U5.3 (EN)
- new net EN_4: R7.1, U2.7 (P3), U6.3 (EN)
- new net EN_5: R6.1, U2.6 (P2), U7.3 (EN)
- new net EN_6: R10.1, U2.5 (P1), U8.3 (EN)
- new net P1: U2.4 (P0)
- new net P2: U2.12 (P7)
- new net VCC: C2.1, R3.1, R4.1, U2.16 (VDD), U9.5 (VOUT)
- new net V_CAM_1: J4.1, U4.5 (VOUT)
- new net V_CAM_2: J3.1, U3.5 (VOUT)
- new net V_CAM_3: J5.1, U5.5 (VOUT)
- new net V_CAM_4: J6.1, U8.5 (VOUT)
- new net V_CAM_5: J7.1, U7.5 (VOUT)
- new net V_CAM_6: J8.1, U6.5 (VOUT)
Other:
- note added: "Cut D4 in MCU"
- note added: "Li-Ion charger"
- note removed: "Cut D4"
- moved on the sheet: J1, J2
