File: PCB/CAMERA_ADAPTER/CAMERA_ADAPTER.kicad_sch (KiCad schematic)
At the start: 39 parts, among them J1 Conn_02x06_Odd_Even, J2 Conn_02x06_Odd_Even, J3 BM06B-SRSS-TBT(LF)(SN), J4 BM06B-SRSS-TBT(LF)(SN), J5 BM06B-SRSS-TBT(LF)(SN), J6 BM06B-SRSS-TBT(LF)(SN), J7 BM06B-SRSS-TBT(LF)(SN), J8 BM06B-SRSS-TBT(LF)(SN), J9 Battery, U2 TCA9534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

Commit message: auto stand work
Parts:
- R15: value 1k -> 10k
Changed lines of the file:
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@@
       (effects (font (size 1.27 1.27)))
     )
-    (property "Value" "1k" (at 121.412 165.608 90)
+    (property "Value" "10k" (at 121.412 165.608 90)
       (effects (font (size 1.27 1.27)))
     )
