File: PCB/CAMERA_ADAPTER/CAMERA_ADAPTER.kicad_pcb (KiCad board)
At the start: 2 copper layers, 40 x 46.2 mm, 12 parts, among them J1 Conn_02x06_Odd_Even, J10 Switch, J2 Conn_02x06_Odd_Even, J3 Conn_02x06_Odd_Even

Commit message: udated by FZ
Parts:
- removed D2: LED, LED_SMD:LED_1206_3216Metric_Pad1.42x1.75mm_HandSolder
- removed J10: Switch, Connector_PinHeader_2.00mm:PinHeader_1x02_P2.00mm_Vertical
- removed S1: 500SSP1S2M2QEA, Mylib:SW_500SSP1S2M2QEA
- removed TP1, TP2, TP3, TP4: TestPoint, TestPoint:TestPoint_Pad_1.0x1.0mm
- added C1: 0.1uF, Capacitor_SMD:C_0603_1608Metric_Pad1.08x0.95mm_HandSolder, B.Cu at (151.2, 91.2)
- added C2: 0.1uF, Capacitor_SMD:C_0603_1608Metric_Pad1.08x0.95mm_HandSolder, B.Cu at (146.4, 98.9)
- added C3: 0.1uF, Capacitor_SMD:C_0402_1005Metric_Pad0.74x0.62mm_HandSolder, B.Cu at (142.8, 92.7)
- added C4: 0.1uF, Capacitor_SMD:C_0402_1005Metric_Pad0.74x0.62mm_HandSolder, B.Cu at (140.8, 98.6)
- added C5: 0.1uF, Capacitor_SMD:C_0402_1005Metric_Pad0.74x0.62mm_HandSolder, B.Cu at (159.8, 105.4)
- added C6: 0.1uF, Capacitor_SMD:C_0402_1005Metric_Pad0.74x0.62mm_HandSolder, B.Cu at (140.8, 105.4)
- added C7: 0.1uF, Capacitor_SMD:C_0402_1005Metric_Pad0.74x0.62mm_HandSolder, B.Cu at (162.4, 99.9)
- added C8: 0.1uF, Capacitor_SMD:C_0402_1005Metric_Pad0.74x0.62mm_HandSolder, B.Cu at (162.4, 93.3)
- added C9: 0.1uF, Capacitor_SMD:C_0402_1005Metric_Pad0.74x0.62mm_HandSolder, B.Cu at (151.0, 93.5)
- added J4: BM06B-SRSS-TBT(LF)(SN), Connector_JST:JST_SH_BM06B-SRSS-TB_1x06-1MP_P1.00mm_Vertical, F.Cu at (141.7, 101.0)
- added J5: BM06B-SRSS-TBT(LF)(SN), Connector_JST:JST_SH_BM06B-SRSS-TB_1x06-1MP_P1.00mm_Vertical, F.Cu at (141.7, 107.7)
- added J6: BM06B-SRSS-TBT(LF)(SN), Connector_JST:JST_SH_BM06B-SRSS-TB_1x06-1MP_P1.00mm_Vertical, F.Cu at (158.4, 94.4)
- added J7: BM06B-SRSS-TBT(LF)(SN), Connector_JST:JST_SH_BM06B-SRSS-TB_1x06-1MP_P1.00mm_Vertical, F.Cu at (158.4, 101.0)
- added J8: BM06B-SRSS-TBT(LF)(SN), Connector_JST:JST_SH_BM06B-SRSS-TB_1x06-1MP_P1.00mm_Vertical, F.Cu at (158.4, 107.7)
- added J9: Battery, Connector_PinHeader_2.00mm:PinHeader_1x02_P2.00mm_Vertical, F.Cu at (163.1, 86.5)
- added R10: 10k, Resistor_SMD:R_0402_1005Metric_Pad0.72x0.64mm_HandSolder, B.Cu at (160.9, 96.4)
- added R11: 10k, Resistor_SMD:R_0402_1005Metric_Pad0.72x0.64mm_HandSolder, B.Cu at (151.1, 96.5)
- added R2: 1k, Resistor_SMD:R_0603_1608Metric_Pad0.98x0.95mm_HandSolder, B.Cu at (158.8, 89.2)
- added R3: NC, Resistor_SMD:R_0603_1608Metric_Pad0.98x0.95mm_HandSolder, B.Cu at (146.4, 97.3)
- added R4: NC, Resistor_SMD:R_0603_1608Metric_Pad0.98x0.95mm_HandSolder, B.Cu at (148.9, 98.1)
- added R5: 10k, Resistor_SMD:R_0402_1005Metric_Pad0.72x0.64mm_HandSolder, B.Cu at (140.8, 96.4)
- added R6: 10k, Resistor_SMD:R_0402_1005Metric_Pad0.72x0.64mm_HandSolder, B.Cu at (160.9, 103.2)
- added R7: 10k, Resistor_SMD:R_0402_1005Metric_Pad0.72x0.64mm_HandSolder, B.Cu at (160.9, 109.9)
- added R8: 10k, Resistor_SMD:R_0402_1005Metric_Pad0.72x0.64mm_HandSolder, B.Cu at (140.8, 109.9)
- added R9: 10k, Resistor_SMD:R_0402_1005Metric_Pad0.72x0.64mm_HandSolder, B.Cu at (140.8, 103.2)
- added U1: MCP73831-2-OT, Package_TO_SOT_SMD:SOT-23-5, B.Cu at (154.9, 90.2)
- added U2: TCA9534, Package_SO:TSSOP-16_4.4x5mm_P0.65mm, B.Cu at (150.2, 102.7)
- added U3: AP2112K-3.3, Package_TO_SOT_SMD:SOT-23-5, B.Cu at (140.2, 94.2)
- added U4: AP2112K-3.3, Package_TO_SOT_SMD:SOT-23-5, B.Cu at (140.2, 100.9)
- added U5: AP2112K-3.3, Package_TO_SOT_SMD:SOT-23-5, B.Cu at (140.2, 107.6)
- added U6: AP2112K-3.3, Package_TO_SOT_SMD:SOT-23-5, B.Cu at (159.2, 107.6)
- added U7: AP2112K-3.3, Package_TO_SOT_SMD:SOT-23-5, B.Cu at (159.2, 100.9)
- added U8: AP2112K-3.3, Package_TO_SOT_SMD:SOT-23-5, B.Cu at (159.2, 94.2)
- added U9: AP2112K-3.3, Package_TO_SOT_SMD:SOT-23-5, B.Cu at (148.3, 93.9)
- D1: value LED -> RED; footprint LED_SMD:LED_1206_3216Metric_Pad1.42x1.75mm_HandSolder -> LED_SMD:LED_0603_1608Metric_Pad1.05x0.95mm_HandSolder; moved to B.Cu
- J3: value Conn_02x06_Odd_Even -> BM06B-SRSS-TBT(LF)(SN); footprint Connector_PinHeader_2.54mm:PinHeader_2x06_P2.54mm_Vertical -> Connector_JST:JST_SH_BM06B-SRSS-TB_1x06-1MP_P1.00mm_Vertical
- R1: value 1M -> 1k
- moved D1 11.9 mm to (158.8, 90.8)
- moved R1 9.44 mm to (151.2, 89.3), turned to 0 degrees
- moved J3 7.32 mm to (141.7, 94.4), turned to 0 degrees
Connections:
- D1 pad 2: Net-(D1-A) -> +5V
- J3 pad 1: /BAT_BR -> /V_CAM_2
- J3 pad 2: /A5 -> /MISO
- J3 pad 3: /MISO -> /SCK
- J3 pad 4: /A2 -> /MOSI
- J3 pad 5: /A4 -> /A2
- J3 pad 6: /RXD -> GND
- R1 pad 1: Net-(J10-Pin_1) -> GND
- R1 pad 2: GND -> Net-(U1-PROG)
Routing:
- net /CAM_BAT: track 0.00 -> 79.9 mm
- net /MISO: track 12.4 -> 53.2 mm
- net /SCK: track 12.4 -> 49.7 mm, vias 0 -> 1
- net /MOSI: track 12.4 -> 49.3 mm, vias 0 -> 1
- net /SCL: track 0.00 -> 27.2 mm, vias 0 -> 1
- net /SDA: track 0.00 -> 24.6 mm, vias 0 -> 1
- net /A4: track 16.0 -> 34.4 mm
- net /D12: track 0.00 -> 15.9 mm, vias 0 -> 1
- net +5V: track 0.00 -> 14.8 mm, vias 0 -> 2
- net /RXD: track 13.4 -> 0.00 mm
- net /EN_6: track 0.00 -> 12.7 mm
- net Net-(J10-Pin_1): track 12.4 -> 0.00 mm
- net /BAT_BR: track 12.4 -> 0.00 mm
- net /D2: track 16.0 -> 27.8 mm
- net /EN_1: track 0.00 -> 11.8 mm
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Other:
- outline, holes or cut-outs redrawn
- board text removed: "HexSense Canary Islands"
- board text removed: "ON"
- board text removed: "ResEnv Fangzheng Liu fzliu@mit.edu"

Commit message: udated by FZ
Changed lines of the file:
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@@
     (pad "6" smd roundrect (at 2.5 1.325) (size 0.6 1.55) (layers "F.Cu" "F.Paste" "F.Mask") (roundrect_rratio 0.25)
       (net 1 "GND") (pinfunction "6") (pintype "input"))
-    (pad "MP" smd roundrect (at -3.8 -1.2) (size 1.2 1.8) (layers "F.Cu" "F.Paste" "F.Mask") (roundrect_rratio 0.208333)
-      (net 1 "GND") (pinfunction "MP") (pintype "input"))
-    (pad "MP" smd roundrect (at 3.8 -1.2) (size 1.2 1.8) (layers "F.Cu" "F.Paste" "F.Mask") (roundrect_rratio 0.208333)
+    (pad "MP" smd roundrect (at -3.8 -1.2) (size 1.2 1.8) (layers "F.Cu" "F.Paste" "F.Mask") (roundrect_rratio 0.2083333333)
+      (net 1 "GND") (pinfunction "MP") (pintype "input"))
+    (pad "MP" smd roundrect (at 3.8 -1.2) (size 1.2 1.8) (layers "F.Cu" "F.Paste" "F.Mask") (roundrect_rratio 0.2083333333)
       (net 1 "GND") (pinfunction "MP") (pintype "input"))
     (model ":MYLIB:3D_model/BM06B-SRSS-TBT-LF-SN.STEP"
@@
     (pad "6" smd roundrect (at 2.5 1.325) (size 0.6 1.55) (layers "F.Cu" "F.Paste" "F.Mask") (roundrect_rratio 0.25)
       (net 1 "GND") (pinfunction "6") (pintype "input"))
-    (pad "MP" smd roundrect (at -3.8 -1.2) (size 1.2 1.8) (layers "F.Cu" "F.Paste" "F.Mask") (roundrect_rratio 0.208333)
-      (net 1 "GND") (pinfunction "MP") (pintype "input"))
-    (pad "MP" smd roundrect (at 3.8 -1.2) (size 1.2 1.8) (layers "F.Cu" "F.Paste" "F.Mask") (roundrect_rratio 0.208333)
+    (pad "MP" smd roundrect (at -3.8 -1.2) (size 1.2 1.8) (layers "F.Cu" "F.Paste" "F.Mask") (roundrect_rratio 0.2083333333)
+      (net 1 "GND") (pinfunction "MP") (pintype "input"))
+    (pad "MP" smd roundrect (at 3.8 -1.2) (size 1.2 1.8) (layers "F.Cu" "F.Paste" "F.Mask") (roundrect_rratio 0.2083333333)
       (net 1 "GND") (pinfunction "MP") (pintype "input"))
     (model ":MYLIB:3D_model/BM06B-SRSS-TBT-LF-SN.STEP"
@@
     (pad "6" smd roundrect (at 2.5 1.325) (size 0.6 1.55) (layers "F.Cu" "F.Paste" "F.Mask") (roundrect_rratio 0.25)
       (net 1 "GND") (pinfunction "6") (pintype "input"))
-    (pad "MP" smd roundrect (at -3.8 -1.2) (size 1.2 1.8) (layers "F.Cu" "F.Paste" "F.Mask") (roundrect_rratio 0.208333)
-      (net 1 "GND") (pinfunction "MP") (pintype "input"))
-    (pad "MP" smd roundrect (at 3.8 -1.2) (size 1.2 1.8) (layers "F.Cu" "F.Paste" "F.Mask") (roundrect_rratio 0.208333)
+    (pad "MP" smd roundrect (at -3.8 -1.2) (size 1.2 1.8) (layers "F.Cu" "F.Paste" "F.Mask") (roundrect_rratio 0.2083333333)
+      (net 1 "GND") (pinfunction "MP") (pintype "input"))
+    (pad "MP" smd roundrect (at 3.8 -1.2) (size 1.2 1.8) (layers "F.Cu" "F.Paste" "F.Mask") (roundrect_rratio 0.2083333333)
       (net 1 "GND") (pinfunction "MP") (pintype "input"))
     (model ":MYLIB:3D_model/BM06B-SRSS-TBT-LF-SN.STEP"
@@
     (pad "6" smd roundrect (at 2.5 1.325) (size 0.6 1.55) (layers "F.Cu" "F.Paste" "F.Mask") (roundrect_rratio 0.25)
       (net 1 "GND") (pinfunction "6") (pintype "input"))
-    (pad "MP" smd roundrect (at -3.8 -1.2) (size 1.2 1.8) (layers "F.Cu" "F.Paste" "F.Mask") (roundrect_rratio 0.208333)
-      (net 1 "GND") (pinfunction "MP") (pintype "input"))
-    (pad "MP" smd roundrect (at 3.8 -1.2) (size 1.2 1.8) (layers "F.Cu" "F.Paste" "F.Mask") (roundrect_rratio 0.208333)
+    (pad "MP" smd roundrect (at -3.8 -1.2) (size 1.2 1.8) (layers "F.Cu" "F.Paste" "F.Mask") (roundrect_rratio 0.2083333333)
+      (net 1 "GND") (pinfunction "MP") (pintype "input"))
+    (pad "MP" smd roundrect (at 3.8 -1.2) (size 1.2 1.8) (layers "F.Cu" "F.Paste" "F.Mask") (roundrect_rratio 0.2083333333)
       (net 1 "GND") (pinfunction "MP") (pintype "input"))
     (model ":MYLIB:3D_model/BM06B-SRSS-TBT-LF-SN.STEP"
@@
     (pad "6" smd roundrect (at 2.5 1.325) (size 0.6 1.55) (layers "F.Cu" "F.Paste" "F.Mask") (roundrect_rratio 0.25)
       (net 1 "GND") (pinfunction "6") (pintype "input"))
-    (pad "MP" smd roundrect (at -3.8 -1.2) (size 1.2 1.8) (layers "F.Cu" "F.Paste" "F.Mask") (roundrect_rratio 0.208333)
-      (net 1 "GND") (pinfunction "MP") (pintype "input"))
-    (pad "MP" smd roundrect (at 3.8 -1.2) (size 1.2 1.8) (layers "F.Cu" "F.Paste" "F.Mask") (roundrect_rratio 0.208333)
+    (pad "MP" smd roundrect (at -3.8 -1.2) (size 1.2 1.8) (layers "F.Cu" "F.Paste" "F.Mask") (roundrect_rratio 0.2083333333)
+      (net 1 "GND") (pinfunction "MP") (pintype "input"))
+    (pad "MP" smd roundrect (at 3.8 -1.2) (size 1.2 1.8) (layers "F.Cu" "F.Paste" "F.Mask") (roundrect_rratio 0.2083333333)
       (net 1 "GND") (pinfunction "MP") (pintype "input"))
     (model ":MYLIB:3D_model/BM06B-SRSS-TBT-LF-SN.STEP"
@@
     (pad "6" smd roundrect (at 2.5 1.325) (size 0.6 1.55) (layers "F.Cu" "F.Paste" "F.Mask") (roundrect_rratio 0.25)
       (net 1 "GND") (pinfunction "6") (pintype "input"))
-    (pad "MP" smd roundrect (at -3.8 -1.2) (size 1.2 1.8) (layers "F.Cu" "F.Paste" "F.Mask") (roundrect_rratio 0.208333)
-      (net 1 "GND") (pinfunction "MP") (pintype "input"))
-    (pad "MP" smd roundrect (at 3.8 -1.2) (size 1.2 1.8) (layers "F.Cu" "F.Paste" "F.Mask") (roundrect_rratio 0.208333)
+    (pad "MP" smd roundrect (at -3.8 -1.2) (size 1.2 1.8) (layers "F.Cu" "F.Paste" "F.Mask") (roundrect_rratio 0.2083333333)
+      (net 1 "GND") (pinfunction "MP") (pintype "input"))
+    (pad "MP" smd roundrect (at 3.8 -1.2) (size 1.2 1.8) (layers "F.Cu" "F.Paste" "F.Mask") (roundrect_rratio 0.2083333333)
       (net 1 "GND") (pinfunction "MP") (pintype "input"))
     (model ":MYLIB:3D_model/BM06B-SRSS-TBT-LF-SN.STEP"

Commit message: auto stand work
Parts:
- R1: value 1k -> 10k
Connections:
- net /RXD renamed /LoRa_CS
Changed lines of the file:
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@@
   (net 5 "/A5")
   (net 6 "/VBAT")
-  (net 7 "/RXD")
+  (net 7 "/LoRa_CS")
   (net 8 "/BURN_EN")
   (net 9 "/A3")
@@
       (net 12 "/A2") (pinfunction "Pin_6") (pintype "passive"))
     (pad "7" thru_hole oval (at 0 7.62 90) (size 1.7 1.7) (drill 1) (layers "*.Cu" "*.Mask")
-      (net 7 "/RXD") (pinfunction "Pin_7") (pintype "passive"))
+      (net 7 "/LoRa_CS") (pinfunction "Pin_7") (pintype "passive"))
     (pad "8" thru_hole oval (at 2.54 7.62 90) (size 1.7 1.7) (drill 1) (layers "*.Cu" "*.Mask")
       (net 1 "GND") (pinfunction "Pin_8") (pintype "passive"))
@@
         (effects (font (size 1 1) (thickness 0.15)) (justify mirror))
     )
-    (fp_text value "1k" (at 0 -1.43) (layer "B.Fab")
-        (effects (font (size 1 1) (thickness 0.15)) (justify mirror))
-    )
+    (fp_text value "10k" (at 0 -1.43) (layer "B.Fab")
+        (effects (font (size 1 1) (thickness 0.15)) (justify mirror))
+    )
