File: PCB/CONN/CONN.kicad_sch (KiCad schematic)
At the start: 12 parts, among them J1 Conn_02x06_Odd_Even, J10 Switch, J2 Conn_02x06_Odd_Even, J3 Conn_02x06_Odd_Even

Commit message: udated by FZ
Other:
- note added: "Cut D4 in MCU"
- note removed: "Cut D4"
Changed lines of the file:
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@@
   )
   (no_connect (at 193.04 49.53))
+  (polyline (pts (xy 156.21 101.6) (xy 171.958 101.6))
+    (stroke (width 0) (type default))
+  )
   (wire (pts (xy 194.31 127) (xy 200.66 127))
     (stroke (width 0) (type default))
@@
     (stroke (width 0) (type default))
   )
-  (polyline (pts (xy 163.195 100.965) (xy 171.45 100.965))
-    (stroke (width 0) (type default))
-  )
   (wire (pts (xy 186.69 36.83) (xy 186.69 38.1))
     (stroke (width 0) (type default))
@@
     (stroke (width 0) (type default))
   )
-  (polyline (pts (xy 171.45 104.14) (xy 163.195 104.14))
-    (stroke (width 0) (type default))
-  )
   (wire (pts (xy 175.26 46.99) (xy 175.26 38.1))
     (stroke (width 0) (type default))
@@
     (stroke (width 0) (type default))
   )
+  (polyline (pts (xy 156.21 101.6) (xy 156.21 104.775))
+    (stroke (width 0) (type default))
+  )
   (polyline (pts (xy 134.62 13.97) (xy 240.03 13.97))
     (stroke (width 0) (type default))
@@
     (stroke (width 0) (type default))
   )
-  (polyline (pts (xy 171.45 100.965) (xy 171.45 104.14))
+  (polyline (pts (xy 171.958 104.775) (xy 156.21 104.775))
     (stroke (width 0) (type default))
   )
@@
     (stroke (width 0) (type default))
   )
+  (polyline (pts (xy 171.958 101.6) (xy 171.958 104.648))
+    (stroke (width 0) (type default))
+  )
   (wire (pts (xy 194.31 72.39) (xy 203.2 72.39))
     (stroke (width 0) (type default))
@@
     (stroke (width 0) (type default))
   )
-  (polyline (pts (xy 163.195 100.965) (xy 163.195 104.14))
-    (stroke (width 0) (type default))
-  )
   (wire (pts (xy 172.72 96.52) (xy 181.61 96.52))
     (stroke (width 0) (type default))
@@
   (wire (pts (xy 194.31 119.38) (xy 200.66 119.38))
     (stroke (width 0) (type default))
-  )
-  (text "Cut D4" (at 163.83 103.632 0)
-    (effects (font (size 1.27 1.27)) (justify left bottom))
   )
   (text "Connector" (at 138.43 21.59 0)
     (effects (font (size 3 3) (thickness 0.508) bold) (justify left bottom))
   )
+  (text "Cut D4 in MCU" (at 156.718 104.14 0)
+    (effects (font (size 1.27 1.27)) (justify left bottom))
+  )
   (label "D3" (at 203.2 96.52 180) (fields_autoplaced)
     (effects (font (size 1.27 1.27)) (justify right bottom))
@@
     (effects (font (size 1.27 1.27)) (justify right bottom))
   )
+  (label "LORA_FREQ_SELECT" (at 203.2 91.44 0) (fields_autoplaced)
+    (effects (font (size 1.27 1.27)) (justify left bottom))
+  )
   (label "SCK" (at 172.72 127 0) (fields_autoplaced)
