File: PCB/BURNING_R/V1/BURNING_R.kicad_sch (KiCad schematic)
At the start: 36 parts, among them J1 Conn_02x06_Odd_Even, J10 Switch, J2 Conn_02x06_Odd_Even, J3 BR_conn, J4 BR_conn, J5 BR_conn, J6 BR_conn, J7 BR_conn, J8 BR_conn, J9 Battery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

Commit message: udated by FZ
Other:
- note added: "Cut D4 in MCU"
- note removed: "Cut D4"
Changed lines of the file:
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@@
     (stroke (width 0) (type default))
   )
-  (polyline (pts (xy 184.785 57.785) (xy 193.04 57.785))
+  (polyline (pts (xy 177.292 57.912) (xy 193.04 57.912))
     (stroke (width 0) (type default))
   )
@@
     (stroke (width 0) (type default))
   )
-  (polyline (pts (xy 193.04 60.96) (xy 184.785 60.96))
+  (polyline (pts (xy 193.04 61.087) (xy 177.292 61.087))
     (stroke (width 0) (type default))
   )
@@
     (stroke (width 0) (type default))
   )
-  (polyline (pts (xy 184.785 57.785) (xy 184.785 60.96))
+  (polyline (pts (xy 177.292 57.912) (xy 177.292 61.087))
     (stroke (width 0) (type default))
   )
@@
     (effects (font (size 2 2) (thickness 0.4) bold) (justify left bottom))
   )
-  (text "Cut D4" (at 185.42 60.452 0)
+  (text "Cut D4 in MCU" (at 177.8 60.452 0)
     (effects (font (size 1.27 1.27)) (justify left bottom))
   )

Commit message: udated by FZ
Parts:
- R16: value 1k -> 10k
Changed lines of the file:
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@@
     (effects (font (size 1.27 1.27)) (justify right bottom))
+  )
+  (label "LORA_FREQ_SELECT" (at 224.79 48.26 0) (fields_autoplaced)
+    (effects (font (size 1.27 1.27)) (justify left bottom))
   )
   (label "VBUS" (at 163.83 30.48 180) (fields_autoplaced)
@@
       (effects (font (size 1.27 1.27)))
     )
-    (property "Value" "1k" (at 29.21 171.196 90)
+    (property "Value" "10k" (at 29.21 171.196 90)
       (effects (font (size 1.27 1.27)))
     )
