File: PCB/BURNING_R/V1/BURNING_R.kicad_sch (KiCad schematic)
At the start: 36 parts, among them J1 Conn_02x06_Odd_Even, J10 Switch, J2 Conn_02x06_Odd_Even, J3 BR_conn, J4 BR_conn, J5 BR_conn, J6 BR_conn, J7 BR_conn, J8 BR_conn, J9 Battery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

Commit message: auto stand work
Parts:
- R15: value 1k -> 10k
Changed lines of the file:
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@@
       (effects (font (size 1.27 1.27)))
     )
-    (property "Value" "1k" (at 121.412 165.608 90)
+    (property "Value" "10k" (at 121.412 165.608 90)
       (effects (font (size 1.27 1.27)))
     )
