File: PCB/LORA_ADAPTER/LORA_ADAPTER.kicad_pcb (KiCad board)
At the start: 2 copper layers, 40 x 46.2 mm, 39 parts, among them J1 Conn_02x06_Odd_Even, J2 Conn_02x06_Odd_Even, J3 BM06B-SRSS-TBT(LF)(SN), J4 BM06B-SRSS-TBT(LF)(SN), J5 BM06B-SRSS-TBT(LF)(SN), J6 BM06B-SRSS-TBT(LF)(SN), J7 BM06B-SRSS-TBT(LF)(SN), J8 BM06B-SRSS-TBT(LF)(SN), J9 Battery, U1 MCP73831-2-OT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

Commit message: udated by FZ
Parts:
- removed C1, C2: 0.1uF, Capacitor_SMD:C_0603_1608Metric_Pad1.08x0.95mm_HandSolder
- removed C3, C4, C5, C6, C7, C8: 0.1uF, Capacitor_SMD:C_0402_1005Metric_Pad0.74x0.62mm_HandSolder
- removed D1: RED, LED_SMD:LED_0603_1608Metric_Pad1.05x0.95mm_HandSolder
- removed J4, J5, J6, J7, J8: BM06B-SRSS-TBT(LF)(SN), Connector_JST:JST_SH_BM06B-SRSS-TB_1x06-1MP_P1.00mm_Vertical
- removed J9: Battery, Connector_PinHeader_2.00mm:PinHeader_1x02_P2.00mm_Vertical
- removed R10, R11, R5, R6, R7, R8, R9: 10k, Resistor_SMD:R_0402_1005Metric_Pad0.72x0.64mm_HandSolder
- removed R2: 1k, Resistor_SMD:R_0603_1608Metric_Pad0.98x0.95mm_HandSolder
- removed R3, R4: NC, Resistor_SMD:R_0603_1608Metric_Pad0.98x0.95mm_HandSolder
- removed U1: MCP73831-2-OT, Package_TO_SOT_SMD:SOT-23-5
- removed U2: TCA9534, Package_SO:TSSOP-16_4.4x5mm_P0.65mm
- removed U3, U4, U5, U6, U7, U8: AP2112K-3.3, Package_TO_SOT_SMD:SOT-23-5
- added S1: 500SSP1S2M2QEA, Mylib:SW_500SSP1S2M2QEA, F.Cu at (138.2, 99.7)
- C9, U9: moved to F.Cu
- J3: value BM06B-SRSS-TBT(LF)(SN) -> SM06B-SRSS-TB(LF)(SN); footprint Connector_JST:JST_SH_BM06B-SRSS-TB_1x06-1MP_P1.00mm_Vertical -> Connector_JST:JST_SH_SM06B-SRSS-TB_1x06-1MP_P1.00mm_Horizontal
- R1: value 1k -> 10k; footprint Resistor_SMD:R_0603_1608Metric_Pad0.98x0.95mm_HandSolder -> Resistor_SMD:R_0402_1005Metric_Pad0.72x0.64mm_HandSolder; moved to F.Cu
- moved J3 11.4 mm to (151.5, 100.1), turned to 90 degrees
- moved R1 8.17 mm to (144.8, 94.4), turned to 180 degrees
- moved C9 8.05 mm to (143.3, 91.2), turned to 180 degrees
- moved U9 2.55 mm to (146.6, 92.1), turned to 0 degrees
Connections:
- C9 pad 1: /CAM_BAT -> /VBAT
- J1 pad 7: /RXD -> /LoRa_CS
- J3 pad 1: /V_CAM_2 -> GND
- J3 pad 5: /A2 -> /LoRa_CS
- J3 pad 6: GND -> +3V3
- R1 pad 1: GND -> /A3
- R1 pad 2: Net-(U1-PROG) -> GND
- U9 pad 1: /CAM_BAT -> /VBAT
- U9 pad 3: /A4 -> /A3
- U9 pad 5: VCC -> +3V3
Routing:
- net /CAM_BAT: track 79.9 -> 0.00 mm
- net /MISO: track 53.2 -> 14.1 mm
- net /SCK: track 49.7 -> 14.7 mm, vias 1 -> 0
- net /A4: track 34.4 -> 0.00 mm
- net /MOSI: track 49.3 -> 16.8 mm, vias 1 -> 0
- net /D2: track 27.8 -> 0.00 mm
- net /SCL: track 27.2 -> 0.00 mm, vias 1 -> 0
- net /SDA: track 24.6 -> 0.00 mm, vias 1 -> 0
- net /D1: track 23.0 -> 0.00 mm
- net /A5: track 18.1 -> 0.00 mm
- net /D12: track 15.9 -> 0.00 mm, vias 1 -> 0
- net /A2: track 15.2 -> 0.00 mm
- net +5V: track 14.8 -> 0.00 mm, vias 2 -> 0
- net /LoRa_CS: track 0.00 -> 13.5 mm
- net /D3: track 13.4 -> 0.00 mm
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Other:
- outline, holes or cut-outs redrawn

Commit message: udated by FZ
Parts:
- added J4: Battery, Connector_PinHeader_2.54mm:PinHeader_1x02_P2.54mm_Vertical, F.Cu at (132.7, 101.3)
Connections:
- S1 pad 1: unconnected-(S1-Pad1) -> Net-(J4-Pin_1)
- S1 pad 2: unconnected-(S1-Pad2) -> Net-(J4-Pin_2)
Routing:
- net Net-(J4-Pin_1): track 0.00 -> 6.85 mm
- net Net-(J4-Pin_2): track 0.00 -> 5.95 mm
- net GND: vias 119 -> 114
Other:
- outline, holes or cut-outs redrawn
- board text added: "ON"
