File: PCB/LORA_ADAPTER/LORA_ADAPTER.kicad_sch (KiCad schematic)
At the start: 39 parts, among them J1 Conn_02x06_Odd_Even, J2 Conn_02x06_Odd_Even, J3 BM06B-SRSS-TBT(LF)(SN), J4 BM06B-SRSS-TBT(LF)(SN), J5 BM06B-SRSS-TBT(LF)(SN), J6 BM06B-SRSS-TBT(LF)(SN), J7 BM06B-SRSS-TBT(LF)(SN), J8 BM06B-SRSS-TBT(LF)(SN), J9 Battery, U2 TCA9534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

Commit message: udated by FZ
Other:
- moved on the sheet: C2, C3, C4, C5, C6, C7, C8, C9, J9, R10, R11, R4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

Commit message: udated by FZ
Parts:
- removed C13, C2: 0.1uF, Capacitor_SMD:C_0603_1608Metric_Pad1.08x0.95mm_HandSolder, symbol Device:C_Small
- removed C3, C4, C5, C6, C7, C8: 0.1uF, Capacitor_SMD:C_0402_1005Metric_Pad0.74x0.62mm_HandSolder, symbol Device:C_Small
- removed D1: RED, LED_SMD:LED_0603_1608Metric_Pad1.05x0.95mm_HandSolder, symbol Device:LED_Small_Filled
- removed J4, J5, J6, J7, J8: BM06B-SRSS-TBT(LF)(SN), Connector_JST:JST_SH_BM06B-SRSS-TB_1x06-1MP_P1.00mm_Vertical, symbol Mylib:BM06B-SURS-TF(LF)(SN)
- removed J9: Battery, Connector_PinHeader_2.00mm:PinHeader_1x02_P2.00mm_Vertical, symbol Connector:Conn_01x02_Pin
- removed R10, R11, R5, R6, R7, R8, R9: 10k, Resistor_SMD:R_0402_1005Metric_Pad0.72x0.64mm_HandSolder, symbol Device:R_Small
- removed R15, R16: 1k, Resistor_SMD:R_0603_1608Metric_Pad0.98x0.95mm_HandSolder, symbol Device:R_Small
- removed R3, R4: NC, Resistor_SMD:R_0603_1608Metric_Pad0.98x0.95mm_HandSolder, symbol Device:R_Small
- removed U2: TCA9534, Package_SO:TSSOP-16_4.4x5mm_P0.65mm, symbol Interface_Expansion:TCA9534
- removed U3, U4, U5, U6, U7, U8: AP2112K-3.3, Package_TO_SOT_SMD:SOT-23-5, symbol Regulator_Linear:AP2112K-3.3
- removed U4: MCP73831-2-OT, Package_TO_SOT_SMD:SOT-23-5, symbol Battery_Management:MCP73831-2-OT
- added R1: 10k, Resistor_SMD:R_0402_1005Metric_Pad0.72x0.64mm_HandSolder, symbol Device:R_Small
- added S1: 500SSP1S2M2QEA, Mylib:SW_500SSP1S2M2QEA, symbol 500SSP1S2M2QEA:500SSP1S2M2QEA
- J3: value BM06B-SRSS-TBT(LF)(SN) -> SM06B-SRSS-TB(LF)(SN); footprint Connector_JST:JST_SH_BM06B-SRSS-TB_1x06-1MP_P1.00mm_Vertical -> Connector_JST:JST_SH_SM06B-SRSS-TB_1x06-1MP_P1.00mm_Horizontal
Connections:
- net CAM_BAT is gone; now on net VBAT: C9.1, U9.1 (VIN)
- net V_CAM_2 is gone; now on net GND: J3.1
- net A2: no longer J3.5
- net A3: now also U9.3 (EN), R1.1
- net A4: no longer U9.3 (EN)
- net GND: now also R1.2; no longer J3.6
- net LoRa_CS: now also J3.5
- net VCC renamed +3V3
- net +3V3: now also J3.6
- no-connect marks 1 -> 0
Other:
- note removed: "Li-Ion charger"
- moved on the sheet: J1, J2

Commit message: udated by FZ
Parts:
- added J4: Battery, Connector_PinHeader_2.54mm:PinHeader_1x02_P2.54mm_Vertical, symbol Connector:Conn_01x02_Pin
Connections:
- net at S1.1: now also J4.1 (Pin_1)
- net at S1.2: now also J4.2 (Pin_2)
Changed lines of the file:
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@@
+    (stroke (width 0) (type default))
+  )
+  (wire (pts (xy 67.31 67.31) (xy 67.31 68.58))
     (stroke (width 0) (type default))
   )
@@
     (stroke (width 0) (type default))
   )
+  (wire (pts (xy 64.77 68.58) (xy 64.77 67.31))
+    (stroke (width 0) (type default))
+  )
   (wire (pts (xy 91.44 35.56) (xy 91.44 38.1))
     (stroke (width 0) (type default))
@@
     (stroke (width 0) (type default))
   )
+  (wire (pts (xy 59.69 77.47) (xy 54.61 77.47))
+    (stroke (width 0) (type default))
+  )
   (wire (pts (xy 175.26 120.65) (xy 182.88 120.65))
     (stroke (width 0) (type default))
@@
     (stroke (width 0) (type default))
   )
+  (wire (pts (xy 80.01 74.93) (xy 74.93 74.93))
+    (stroke (width 0) (type default))
+  )
   (wire (pts (xy 181.61 110.49) (xy 182.88 110.49))
     (stroke (width 0) (type default))
@@
     (stroke (width 0) (type default))
   )
+  (wire (pts (xy 67.31 68.58) (xy 80.01 68.58))
+    (stroke (width 0) (type default))
+  )
+  (wire (pts (xy 80.01 68.58) (xy 80.01 74.93))
+    (stroke (width 0) (type default))
+  )
   (wire (pts (xy 195.58 113.03) (xy 195.58 114.3))
     (stroke (width 0) (type default))
@@
     (stroke (width 0) (type default))
   )
+  (wire (pts (xy 54.61 68.58) (xy 64.77 68.58))
+    (stroke (width 0) (type default))
+  )
   (polyline (pts (xy 173.228 80.645) (xy 157.48 80.645))
+    (stroke (width 0) (type default))
+  )
+  (wire (pts (xy 54.61 77.47) (xy 54.61 68.58))
     (stroke (width 0) (type default))
   )
@@
         )
       )
+    )
+  )
+  (symbol (lib_id "Connector:Conn_01x02_Pin") (at 67.31 62.23 270) (unit 1)
+    (in_bom yes) (on_board yes) (dnp no) (fields_autoplaced)
+    (property "Reference" "J4" (at 68.1482 61.841 90)
+      (effects (font (size 1.27 1.27)) (justify left))
+    )
+    (property "Value" "Battery" (at 68.1482 63.889 90)
+      (effects (font (size 1.27 1.27)) (justify left))
+    )
+    (property "Footprint" "Connector_PinHeader_2.54mm:PinHeader_1x02_P2.54mm_Vertical" (at 67.31 62.23 0)
+      (effects (font (size 1.27 1.27)) hide)
+    )
+    (property "Datasheet" "~" (at 67.31 62.23 0)
+      (effects (font (size 1.27 1.27)) hide)
+    )
+    (pin "1")
+    (pin "2")
+    (instances
+      (project "LORA_ADAPTER"
+        (path "/e63e39d7-6ac0-4ffd-8aa3-1841a4541b55"
+          (reference "J4") (unit 1)
+        )
+      )

Commit message: udated by FZ
Other:
- note added: "Cut DCDC_EN in LoRa_adapter"
Changed lines of the file:
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@@
+    (stroke (width 0) (type default))
+  )
+  (polyline (pts (xy 83.82 22.86) (xy 83.82 26.543))
     (stroke (width 0) (type default))
   )
@@
     (stroke (width 0) (type default))
   )
+  (polyline (pts (xy 228.6 38.1) (xy 196.85 38.1))
+    (stroke (width 0) (type default))
+  )
   (wire (pts (xy 64.77 68.58) (xy 64.77 67.31))
     (stroke (width 0) (type default))
@@
     (stroke (width 0) (type default))
   )
+  (polyline (pts (xy 83.82 26.67) (xy 52.07 26.67))
+    (stroke (width 0) (type default))
+  )
   (polyline (pts (xy 173.228 77.47) (xy 173.228 80.518))
     (stroke (width 0) (type default))
@@
     (stroke (width 0) (type default))
   )
+  (polyline (pts (xy 196.85 34.29) (xy 196.85 38.1))
+    (stroke (width 0) (type default))
+  )
   (wire (pts (xy 173.99 69.85) (xy 182.88 69.85))
     (stroke (width 0) (type default))
   )
+  (polyline (pts (xy 196.85 34.29) (xy 228.6 34.29))
+    (stroke (width 0) (type default))
+  )
   (wire (pts (xy 195.58 110.49) (xy 195.58 113.03))
     (stroke (width 0) (type default))
@@
     (stroke (width 0) (type default))
   )
+  (wire (pts (xy 87.63 30.48) (xy 91.44 30.48))
+    (stroke (width 0) (type default))
+  )
   (wire (pts (xy 181.61 110.49) (xy 182.88 110.49))
     (stroke (width 0) (type default))
   )
+  (polyline (pts (xy 52.07 22.86) (xy 83.82 22.86))
+    (stroke (width 0) (type default))
+  )
   (wire (pts (xy 184.15 31.75) (xy 194.31 31.75))
     (stroke (width 0) (type default))
@@
     (stroke (width 0) (type default))
   )
+  (polyline (pts (xy 52.07 22.86) (xy 52.07 26.67))
+    (stroke (width 0) (type default))
+  )
   (wire (pts (xy 195.58 43.18) (xy 204.47 43.18))
     (stroke (width 0) (type default))
@@
     (stroke (width 0) (type default))
   )
+  (polyline (pts (xy 228.6 34.29) (xy 228.6 37.973))
+    (stroke (width 0) (type default))
+  )
   (wire (pts (xy 195.58 45.72) (xy 204.47 45.72))
     (stroke (width 0) (type default))
@@
     (stroke (width 0) (type default))
   )
-  (wire (pts (xy 91.44 29.21) (xy 95.25 29.21))
+  (wire (pts (xy 87.63 29.21) (xy 95.25 29.21))
     (stroke (width 0) (type default))
   )
@@
     (stroke (width 0) (type default))
   )
-  (wire (pts (xy 91.44 29.21) (xy 91.44 30.48))
+  (wire (pts (xy 87.63 29.21) (xy 87.63 30.48))
     (stroke (width 0) (type default))
   )
@@
     (effects (font (size 3 3) (thickness 0.508) bold) (justify left bottom))
   )
+  (text "Cut DCDC_EN in LoRa_adapter" (at 198.12 37.465 0)
+    (effects (font (size 1.27 1.27)) (justify left bottom))
+  )
+  (text "Cut DCDC_EN in LoRa_adapter" (at 53.34 26.035 0)
+    (effects (font (size 1.27 1.27)) (justify left bottom))
+  )
   (label "D3" (at 204.47 72.39 180) (fields_autoplaced)
     (effects (font (size 1.27 1.27)) (justify right bottom))
@@
     (effects (font (size 1.27 1.27)) (justify left bottom))
   )
-  (label "A3" (at 91.44 29.21 0) (fields_autoplaced)
+  (label "DCDC_EN" (at 87.63 29.21 0) (fields_autoplaced)
     (effects (font (size 1.27 1.27)) (justify left bottom))
   )
@@
     (effects (font (size 1.27 1.27)) (justify left bottom))
   )
+  (label "DCDC_EN" (at 204.47 45.72 0) (fields_autoplaced)
+    (effects (font (size 1.27 1.27)) (justify left bottom))
+  )
