File: PCB/LORA/V1/LORA.kicad_pcb (KiCad board)
At the start: 2 copper layers, 40 x 46.2 mm, 15 parts, among them J1 Conn_02x06_Odd_Even, J2 Conn_02x06_Odd_Even, J3 Battery, Q1 NMOS, SW1 SW_SPDT, U1 RFM95CW

Commit message: udated by FZ
Parts:
- removed Q1: NMOS, Package_TO_SOT_SMD:SOT-23
- removed R1: 100, Resistor_SMD:R_0603_1608Metric_Pad0.98x0.95mm_HandSolder
- removed R2: 10k, Resistor_SMD:R_0603_1608Metric_Pad0.98x0.95mm_HandSolder
- removed SW1: SW_SPDT, Connector_PinHeader_2.54mm:PinHeader_1x03_P2.54mm_Vertical
- added D4: LED, LED_SMD:LED_0603_1608Metric_Pad1.05x0.95mm_HandSolder, F.Cu at (167.7, 98.7)
- added J4: BM06B-SRSS-TBT(LF)(SN), Connector_JST:JST_SH_BM06B-SRSS-TB_1x06-1MP_P1.00mm_Vertical, B.Cu at (161.5, 100.0)
- added J5: Conn_01x02_Pin, Connector_PinHeader_2.00mm:PinHeader_1x02_P2.00mm_Vertical, F.Cu at (167.6, 101.7)
- added J6: Conn_01x02_Pin, Connector_PinHeader_2.00mm:PinHeader_1x02_P2.00mm_Vertical, F.Cu at (162.2, 89.9)
- C1: value 47uF -> 10uF; footprint Capacitor_Tantalum_SMD:CP_EIA-6032-15_Kemet-U_Pad2.25x2.35mm_HandSolder -> Capacitor_SMD:C_1206_3216Metric_Pad1.33x1.80mm_HandSolder; moved to B.Cu
- C2: value 10uF -> 0.1uF; moved to B.Cu
- D1, D2, D3: footprint LED_SMD:LED_1206_3216Metric_Pad1.42x1.75mm_HandSolder -> LED_SMD:LED_0603_1608Metric_Pad1.05x0.95mm_HandSolder
- J3: value Battery -> BM06B-SRSS-TBT(LF)(SN); footprint Connector_PinHeader_2.54mm:PinHeader_1x02_P2.54mm_Vertical -> Connector_JST:JST_SH_BM06B-SRSS-TB_1x06-1MP_P1.00mm_Vertical; moved to B.Cu
- moved C1 21.0 mm to (143.6, 103.4)
- moved D1 18.3 mm to (167.7, 95.5), turned to 0 degrees
- moved D2 15.0 mm to (167.7, 97.1), turned to 0 degrees
- moved C2 14.2 mm to (152.1, 104.1), turned to -90 degrees
- moved J3 12.3 mm to (156.2, 100.0), turned to -90 degrees
- moved D3 1.60 mm to (162.0, 87.5), turned to 0 degrees
- moved R3 1.53 mm to (155.4, 90.9)
Connections:
- net +5V renamed /A2
- net /D11 renamed /D12
- net /D13 renamed /D10
- net /D6 renamed /D1
- net /~{EN} renamed /D8
- net /~{I2C_RESET} renamed /VBUS
- C1 pad 1: /VBAT1 -> VCC
- D1 pad 1: /CHG2- -> /LED02
- D1 pad 2: /CHG2+ -> /LED01
- D2 pad 1: /CHG1- -> /LED12
- D2 pad 2: /CHG1+ -> /LED11
- D3 pad 1: Net-(D3-K) -> /LED32
- D3 pad 2: Net-(D3-A) -> /LED31
- J1 pad 3: VCC -> /A5
- J1 pad 4: /VBAT_OK -> /A3
- J1 pad 7: /RXD -> /LoRa_CS
- J1 pad 9: /TXD -> /BURN_EN
- J2 pad 11: /LED2 -> /BAT_BR
- J2 pad 3: /A1 -> /MOSI
- J2 pad 6: /A5 -> /D3
- J2 pad 7: /MOSI -> /D2
- J2 pad 8: /~{CS} -> /A4
- J3 pad 1: /MAIN_BAT -> GND
- J3 pad 2: /VBAT1 -> /MISO
- U1 pad 13: /~{CS} -> /LoRa_CS
- U1 pad 6: unconnected-(U1-DIO0-Pad6) -> /A3
Routing:
- net /A3: track 0.00 -> 48.9 mm, vias 0 -> 1
- net /LoRa_CS: track 0.00 -> 22.6 mm, vias 0 -> 1
- net /~{CS}: track 21.3 -> 0.00 mm
- net /MISO: track 18.0 -> 32.6 mm
- net /TXD: track 14.1 -> 0.00 mm
- net /RST_LoRa: track 11.0 -> 21.4 mm
- net /MAIN_BAT: track 8.30 -> 0.00 mm
- net /VBAT1: track 8.16 -> 0.00 mm
- net /LED21: track 0.00 -> 7.32 mm, vias 0 -> 1
- net /LED11: track 0.00 -> 7.16 mm, vias 0 -> 1
- net /LED01: track 0.00 -> 7.00 mm, vias 0 -> 1
- net Net-(D3-K): track 6.08 -> 0.00 mm
- net /LED22: track 0.00 -> 5.16 mm, vias 0 -> 1
- net /LED12: track 0.00 -> 4.99 mm, vias 0 -> 1
- net /LED02: track 0.00 -> 4.83 mm, vias 0 -> 1
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